Commit message: Task O

File: ball.urdf (robot description, URDF)
Before this commit: robot robot, 1 links, 0 joints
Links:
- link tempBall: geometry collision box size=0.5 0.5 0.5; visual box size=0.5 0.5 0.5

File: body.urdf (robot description, URDF)
Before this commit: robot robot, 7 links, 6 joints
Joints:
- joint Torso_Link1: origin xyz=0 0.5 0.5 rpy=0 0 0 -> xyz=0 0 0.25 rpy=0 0 0
