Commit message: etc

File: body 2.urdf (robot description, URDF)
Before this commit: robot robot, 12 links, 11 joints
Links:
- removed link Link10
- link Link0: geometry collision box size=0.7042927395452226 0.4468405807395923 0.5377907003560002; visual box size=0.7042927395452226 0.4468405807395923 0.5377907003560002
- link Link1: geometry collision box size=0.22947568673159668 0.1910829720052709 0.756075151088872; visual box size=0.22947568673159668 0.1910829720052709 0.756075151088872
- link Link2: geometry collision box size=0.24523660530945757 0.9438051177941271 0.4896968615802706; visual box size=0.24523660530945757 0.9438051177941271 0.4896968615802706
- link Link3: geometry collision box size=0.9448846439385818 0.47986371128306626 0.46209778163558557; visual box size=0.9448846439385818 0.47986371128306626 0.46209778163558557
- link Link4: geometry collision box size=0.9234272698790281 0.6351507229720808 0.7833997052640607; visual box size=0.9234272698790281 0.6351507229720808 0.7833997052640607
- link Link5: geometry collision box size=0.571863077640325 0.6688630423383253 0.3141280339039879; visual box size=0.571863077640325 0.6688630423383253 0.3141280339039879
- link Link6: geometry collision box size=0.9213360466492199 0.5489822301141292 0.12595222011531915; visual box size=0.9213360466492199 0.5489822301141292 0.12595222011531915
- link Link7: geometry collision box size=0.15048971822964263 0.15282280749868182 0.7699047946553707; visual box size=0.15048971822964263 0.15282280749868182 0.7699047946553707
- link Link8: geometry collision box size=0.5233171461359093 0.41292280493050904 0.5709686956899424; visual box size=0.5233171461359093 0.41292280493050904 0.5709686956899424
- link Link9: geometry collision box size=0.003599801925567858 0.6014371825142077 0.8749022332927467; visual box size=0.003599801925567858 0.6014371825142077 0.8749022332927467
Joints:
- removed joint Link9_Link10
- joint Torso_Link0: origin xyz=0 2.25 0.5 rpy=0 0 0 -> xyz=-3 -3 0.25 rpy=0 0 0
