Commit message: Almost Final Joints Submission
Not sure why the joints are rotating about axis. Will ask prof.

File: body.urdf (robot description, URDF)
Before this commit: robot robot, 4 links, 3 joints
Links:
- removed link Link0
- removed link Link1
- removed link Link2
- removed link Link3
- added link BackLeg, mass 1; collision box size=1 1 1; visual box size=1 1 1
- added link FrontLeg, mass 1; collision box size=1 1 1; visual box size=1 1 1
- added link Torso, mass 1; collision box size=1 1 1; visual box size=1 1 1
Joints:
- removed joint Link0_Link1
- removed joint Link1_Link2
- removed joint Link2_Link3
- added joint Torso_BackLeg: type revolute, parent Torso, child BackLeg, origin xyz=0 1 1 rpy=0 0 0, axis 0 1 0, limit lower=-3.14159 upper=3.14159 effort=0.0 velocity=0.0
- added joint Torso_FrontLeg: type revolute, parent Torso, child FrontLeg, origin xyz=0 2 1 rpy=0 0 0, axis 0 1 0, limit lower=-3.14159 upper=3.14159 effort=0.0 velocity=0.0

Commit message: i broke it

File: body.urdf (robot description, URDF)
Before this commit: robot robot, 9 links, 8 joints
Links:
- removed link BackLeg
- removed link BackLowerLeg
- removed link FrontLowerLeg
- removed link LeftLowerLeg
- removed link RightLeg
- removed link RightLowerLeg
- added link TempBall, mass 1; collision box size=1.5 1.5 1.5; visual box size=1.5 1.5 1.5
- added link Torso_Head, mass 1; collision box size=0.5 0.5 0.5; visual box size=0.5 0.5 0.5
- link LeftLeg: geometry collision box size=0.2 1 0.2; visual box size=0.2 1 0.2
- link Torso: geometry collision box size=2 2 2; visual box size=2 2 2
Joints:
- removed joint BackLeg_BackLowerLeg
- removed joint FrontLeg_FrontLowerLeg
- removed joint LeftLeg_LeftLowerLeg
- removed joint RightLeg_RightLowerLeg
- removed joint Torso_BackLeg
- removed joint Torso_RightLeg
- added joint Torso_Head: type revolute, parent Torso, child Head, origin xyz=-0.5 0 1 rpy=0 0 0, axis 0 1 0, limit lower=-3.14159 upper=3.14159 effort=0.0 velocity=0.0
- joint Torso_FrontLeg: child FrontLeg -> RightLeg; origin xyz=0 0.5 1 rpy=0 0 0 -> xyz=0 3.5 2.0 rpy=0 0 0
- joint Torso_LeftLeg: axis 0 1 0 -> 1 0 0; origin xyz=-0.5 0 1 rpy=0 0 0 -> xyz=0 2.5 2.0 rpy=0 0 0

Commit message: snake attempt, BEFORE WE ADD SPHERES

File: body.urdf (robot description, URDF)
Before this commit: robot robot, 9 links, 8 joints
Links:
- removed link BackLeg
- removed link BackLowerLeg
- removed link FrontLeg
- removed link FrontLowerLeg
- removed link LeftLeg
- removed link LeftLowerLeg
- removed link RightLeg
- removed link RightLowerLeg
- added link Link1, mass 1; collision box size=0.5 0.5 0.5; visual box size=0.5 0.5 0.5
- added link Link2, mass 1; collision box size=0.5 0.5 0.5; visual box size=0.5 0.5 0.5
- added link Link3, mass 1; collision box size=0.5 0.5 0.5; visual box size=0.5 0.5 0.5
- added link Link4, mass 1; collision box size=0.5 0.5 0.5; visual box size=0.5 0.5 0.5
- added link Link5, mass 1; collision box size=0.5 0.5 0.5; visual box size=0.5 0.5 0.5
- added link Link6, mass 1; collision box size=0.5 0.5 0.5; visual box size=0.5 0.5 0.5
- link Torso: geometry collision box size=0.5 0.5 0.5; visual box size=0.5 0.5 0.5
Joints:
- removed joint BackLeg_BackLowerLeg
- removed joint FrontLeg_FrontLowerLeg
- removed joint LeftLeg_LeftLowerLeg
- removed joint RightLeg_RightLowerLeg
- removed joint Torso_BackLeg
- removed joint Torso_FrontLeg
- removed joint Torso_LeftLeg
- removed joint Torso_RightLeg
- added joint Link1_Link2: type revolute, parent Link1, child Link2, origin xyz=0 0.5 0 rpy=0 0 0, axis 1 1 0, limit lower=-3.14159 upper=3.14159 effort=0.0 velocity=0.0
- added joint Link2_Link3: type revolute, parent Link2, child Link3, origin xyz=0 0.5 0 rpy=0 0 0, axis 1 1 0, limit lower=-3.14159 upper=3.14159 effort=0.0 velocity=0.0
- added joint Link3_Link4: type revolute, parent Link3, child Link4, origin xyz=0 0.5 0 rpy=0 0 0, axis 1 1 0, limit lower=-3.14159 upper=3.14159 effort=0.0 velocity=0.0
- added joint Link4_Link5: type revolute, parent Link4, child Link5, origin xyz=0 0.5 0 rpy=0 0 0, axis 1 1 0, limit lower=-3.14159 upper=3.14159 effort=0.0 velocity=0.0
- added joint Link5_Link6: type revolute, parent Link5, child Link6, origin xyz=0 0.5 0 rpy=0 0 0, axis 1 1 0, limit lower=-3.14159 upper=3.14159 effort=0.0 velocity=0.0
- added joint Torso_Link1: type revolute, parent Torso, child Link1, origin xyz=0 0.5 0.5 rpy=0 0 0, axis 1 1 0, limit lower=-3.14159 upper=3.14159 effort=0.0 velocity=0.0

Commit message: Task O Final

File: body.urdf (robot description, URDF)
Before this commit: robot robot, 7 links, 6 joints
Links:
- added link Link7, mass 1; collision box size=0.5 0.5 0.5; visual box size=0.5 0.5 0.5
- added link Link8, mass 1; collision box size=0.35 0.35 0.35; visual box size=0.35 0.35 0.35
- link Link2: geometry collision box size=0.35 0.35 0.35; visual box size=0.35 0.35 0.35
- link Link4: geometry collision box size=0.35 0.35 0.35; visual box size=0.35 0.35 0.35
- link Link6: geometry collision box size=0.35 0.35 0.35; visual box size=0.35 0.35 0.35
Joints:
- added joint Link6_Link7: type revolute, parent Link6, child Link7, origin xyz=0 0.5 0 rpy=0 0 0, axis 1 1 0, limit lower=-3.14159 upper=3.14159 effort=0.0 velocity=0.0
- added joint Link7_Link8: type revolute, parent Link7, child Link8, origin xyz=0 0.5 0 rpy=0 0 0, axis 1 1 0, limit lower=-3.14159 upper=3.14159 effort=0.0 velocity=0.0

Commit message: etc

File: body.urdf (robot description, URDF)
Before this commit: robot robot, 9 links, 8 joints
Links:
- link Link1: geometry collision box size=0.6528696308033384 0.9120362771028819 0.8211606191822324; visual box size=0.6528696308033384 0.9120362771028819 0.8211606191822324
- link Link2: geometry collision box size=0.6471157964915041 0.505275979292136 0.048363974037373025; visual box size=0.6471157964915041 0.505275979292136 0.048363974037373025
- link Link3: geometry collision box size=0.975708300764989 0.34739120527167666 0.3893908793689873; visual box size=0.975708300764989 0.34739120527167666 0.3893908793689873
- link Link4: geometry collision box size=0.8784395385160081 0.8474197846368899 0.29287326373748; visual box size=0.8784395385160081 0.8474197846368899 0.29287326373748
- link Link5: geometry collision box size=0.2591247143425056 0.42494173747944075 0.7606032501063585; visual box size=0.2591247143425056 0.42494173747944075 0.7606032501063585
- link Link6: geometry collision box size=0.6354505221929173 0.314109201650003 0.7303855292709636; visual box size=0.6354505221929173 0.314109201650003 0.7303855292709636
- link Link7: geometry collision box size=0.23878355183452404 0.16051091436447207 0.27178038899076595; visual box size=0.23878355183452404 0.16051091436447207 0.27178038899076595
- link Link8: geometry collision box size=0.2565295750754645 0.48399967065583094 0.07873526155176047; visual box size=0.2565295750754645 0.48399967065583094 0.07873526155176047

Commit message: done

File: body.urdf (robot description, URDF)
Before this commit: robot robot, 9 links, 8 joints
Links:
- link Link1: geometry collision box size=0.17325933398466964 0.2765215132287737 0.6702028114434374; visual box size=0.17325933398466964 0.2765215132287737 0.6702028114434374
- link Link2: geometry collision box size=0.8496752934055971 0.007532149110866748 0.6802631112650475; visual box size=0.8496752934055971 0.007532149110866748 0.6802631112650475
- link Link3: geometry collision box size=0.51213306885312 0.7268987138265174 0.27990623036997053; visual box size=0.51213306885312 0.7268987138265174 0.27990623036997053
- link Link4: geometry collision box size=0.7504889015170103 0.3870096785146693 0.27576479284404565; visual box size=0.7504889015170103 0.3870096785146693 0.27576479284404565
- link Link5: geometry collision box size=0.6437944078487182 0.535780781927006 0.4324188008749972; visual box size=0.6437944078487182 0.535780781927006 0.4324188008749972
- link Link6: geometry collision box size=0.37059798401875144 0.6735949108257318 0.6723719079944156; visual box size=0.37059798401875144 0.6735949108257318 0.6723719079944156
- link Link7: geometry collision box size=0.8937009381794145 0.35559555137769927 0.1396797697120088; visual box size=0.8937009381794145 0.35559555137769927 0.1396797697120088
- link Link8: geometry collision box size=0.0309872599638773 0.30978854850771664 0.11094473470975263; visual box size=0.0309872599638773 0.30978854850771664 0.11094473470975263

Commit message: FINAL DONE!!

File: body.urdf (robot description, URDF)
Before this commit: robot robot, 9 links, 8 joints
Links:
- added link Link0, mass 1; collision box size=0.25035954477062883 0.8515481475687314 0.15966781106368766; visual box size=0.25035954477062883 0.8515481475687314 0.15966781106368766
- added link Link9, mass 1; collision box size=0.37946314607698606 0.21475279496932276 0.16625389930333734; visual box size=0.37946314607698606 0.21475279496932276 0.16625389930333734
- link Link1: geometry collision box size=0.36212837443711354 0.7085540419145717 0.6266498490082001; visual box size=0.36212837443711354 0.7085540419145717 0.6266498490082001
- link Link2: geometry collision box size=0.11906043403904931 0.7595176904843927 0.5839159533663543; visual box size=0.11906043403904931 0.7595176904843927 0.5839159533663543
- link Link3: geometry collision box size=0.5490186187378049 0.784825354970473 0.18351420018615905; visual box size=0.5490186187378049 0.784825354970473 0.18351420018615905
- link Link4: geometry collision box size=0.7337219516013861 0.4335525484633346 0.9282000664982518; visual box size=0.7337219516013861 0.4335525484633346 0.9282000664982518
- link Link5: geometry collision box size=0.8768525055944215 0.27127149212177537 0.24060921535521929; visual box size=0.8768525055944215 0.27127149212177537 0.24060921535521929
- link Link6: geometry collision box size=0.7967796715119219 0.2783063108816871 0.8118541121455675; visual box size=0.7967796715119219 0.2783063108816871 0.8118541121455675
- link Link7: geometry collision box size=0.47144920392114686 0.26741127032680423 0.9846659838018422; visual box size=0.47144920392114686 0.26741127032680423 0.9846659838018422
- link Link8: geometry collision box size=0.28759764059577186 0.8195773308321246 0.8477842117620147; visual box size=0.28759764059577186 0.8195773308321246 0.8477842117620147
Joints:
- removed joint Torso_Link1
- added joint Link0_Link1: type revolute, parent Link0, child Link1, origin xyz=0 0.5 0 rpy=0 0 0, axis 1 1 0, limit lower=-3.14159 upper=3.14159 effort=0.0 velocity=0.0
- added joint Link8_Link9: type revolute, parent Link8, child Link9, origin xyz=0 0.5 0 rpy=0 0 0, axis 1 1 0, limit lower=-3.14159 upper=3.14159 effort=0.0 velocity=0.0
- added joint Torso_Link0: type revolute, parent Torso, child Link0, origin xyz=0 0 0.25 rpy=0 0 0, axis 1 1 0, limit lower=-3.14159 upper=3.14159 effort=0.0 velocity=0.0

Commit message: etc

File: body.urdf (robot description, URDF)
Before this commit: robot robot, 11 links, 10 joints
Links:
- link Link0: geometry collision box size=0.7042927395452226 0.4468405807395923 0.5377907003560002; visual box size=0.7042927395452226 0.4468405807395923 0.5377907003560002
- link Link1: geometry collision box size=0.22947568673159668 0.1910829720052709 0.756075151088872; visual box size=0.22947568673159668 0.1910829720052709 0.756075151088872
- link Link2: geometry collision box size=0.24523660530945757 0.9438051177941271 0.4896968615802706; visual box size=0.24523660530945757 0.9438051177941271 0.4896968615802706
- link Link3: geometry collision box size=0.9448846439385818 0.47986371128306626 0.46209778163558557; visual box size=0.9448846439385818 0.47986371128306626 0.46209778163558557
- link Link4: geometry collision box size=0.9234272698790281 0.6351507229720808 0.7833997052640607; visual box size=0.9234272698790281 0.6351507229720808 0.7833997052640607
- link Link5: geometry collision box size=0.571863077640325 0.6688630423383253 0.3141280339039879; visual box size=0.571863077640325 0.6688630423383253 0.3141280339039879
- link Link6: geometry collision box size=0.9213360466492199 0.5489822301141292 0.12595222011531915; visual box size=0.9213360466492199 0.5489822301141292 0.12595222011531915
- link Link7: geometry collision box size=0.15048971822964263 0.15282280749868182 0.7699047946553707; visual box size=0.15048971822964263 0.15282280749868182 0.7699047946553707
- link Link8: geometry collision box size=0.5233171461359093 0.41292280493050904 0.5709686956899424; visual box size=0.5233171461359093 0.41292280493050904 0.5709686956899424
- link Link9: geometry collision box size=0.003599801925567858 0.6014371825142077 0.8749022332927467; visual box size=0.003599801925567858 0.6014371825142077 0.8749022332927467
Joints:
- joint Torso_Link0: origin xyz=0 0 0.25 rpy=0 0 0 -> xyz=-3 -3 0.25 rpy=0 0 0

Commit message: etc

File: body.urdf (robot description, URDF)
Before this commit: robot robot, 12 links, 11 joints
Links:
- removed link Link10
- removed link Link9
- link Link0: geometry collision box size=0.5517751318653422 0.8962703709689743 0.3540665375815547; visual box size=0.5517751318653422 0.8962703709689743 0.3540665375815547
- link Link1: geometry collision box size=0.01632207201143354 0.017426879615386692 0.6722563570354422; visual box size=0.01632207201143354 0.017426879615386692 0.6722563570354422
- link Link2: geometry collision box size=0.36871696893420547 0.6621633504164444 0.626902371650033; visual box size=0.36871696893420547 0.6621633504164444 0.626902371650033
- link Link3: geometry collision box size=0.6940346628152932 0.9002849590279591 0.2975747619778175; visual box size=0.6940346628152932 0.9002849590279591 0.2975747619778175
- link Link4: geometry collision box size=0.5415986924940379 0.29528233856550523 0.1916421239530527; visual box size=0.5415986924940379 0.29528233856550523 0.1916421239530527
- link Link5: geometry collision box size=0.3871417117157646 0.45900534896959655 0.4314032814880141; visual box size=0.3871417117157646 0.45900534896959655 0.4314032814880141
- link Link6: geometry collision box size=0.5165020736020559 0.15568360255754699 0.10179765048322387; visual box size=0.5165020736020559 0.15568360255754699 0.10179765048322387
- link Link7: geometry collision box size=0.3384106315725034 0.09529451825882185 0.48998675141597114; visual box size=0.3384106315725034 0.09529451825882185 0.48998675141597114
- link Link8: geometry collision box size=0.3306323555961628 0.16279619375486065 0.678857253887734; visual box size=0.3306323555961628 0.16279619375486065 0.678857253887734
Joints:
- removed joint Link8_Link9
- removed joint Link9_Link10

Commit message: etc

File: body.urdf (robot description, URDF)
Before this commit: robot robot, 10 links, 9 joints
Links:
- added link Link10, mass 1; collision box size=0.8633762155215816 0.8535882763581752 0.8318241077348032; visual box size=0.8633762155215816 0.8535882763581752 0.8318241077348032
- added link Link9, mass 1; collision box size=0.08019643178995639 0.28341733832498817 0.8695045253835004; visual box size=0.08019643178995639 0.28341733832498817 0.8695045253835004
- link Link0: geometry collision box size=0.09602739904338886 0.23083563419183806 0.9986216345574274; visual box size=0.09602739904338886 0.23083563419183806 0.9986216345574274
- link Link1: geometry collision box size=0.8332981405054256 0.5871063789828854 0.057844674545931785; visual box size=0.8332981405054256 0.5871063789828854 0.057844674545931785
- link Link2: geometry collision box size=0.07034035524648607 0.14218004457322964 0.22568539355296025; visual box size=0.07034035524648607 0.14218004457322964 0.22568539355296025
- link Link3: geometry collision box size=0.45664171313330404 0.7295379067882815 0.17304619192251236; visual box size=0.45664171313330404 0.7295379067882815 0.17304619192251236
- link Link4: geometry collision box size=0.49995445101046476 0.9818268824835772 0.9152060906398273; visual box size=0.49995445101046476 0.9818268824835772 0.9152060906398273
- link Link5: geometry collision box size=0.24281048124007343 0.424602242129861 0.14972020036268985; visual box size=0.24281048124007343 0.424602242129861 0.14972020036268985
- link Link6: geometry collision box size=0.3998786589315434 0.18403376142715588 0.6332284654271663; visual box size=0.3998786589315434 0.18403376142715588 0.6332284654271663
- link Link7: geometry collision box size=0.595351031328343 0.42608136270384034 0.2580162489756561; visual box size=0.595351031328343 0.42608136270384034 0.2580162489756561
- link Link8: geometry collision box size=0.2543628177896621 0.6780000522780514 0.5692229375994509; visual box size=0.2543628177896621 0.6780000522780514 0.5692229375994509
Joints:
- added joint Link8_Link9: type revolute, parent Link8, child Link9, origin xyz=0 0.5 0 rpy=0 0 0, axis 1 1 0, limit lower=-3.14159 upper=3.14159 effort=0.0 velocity=0.0
- added joint Link9_Link10: type revolute, parent Link9, child Link10, origin xyz=0 0.5 0 rpy=0 0 0, axis 1 1 0, limit lower=-3.14159 upper=3.14159 effort=0.0 velocity=0.0
