Commit message: 2/15/23 OH

File: body.urdf (robot description, URDF)
Before this commit: robot robot, 12 links, 11 joints
Links:
- removed link Link0
- removed link Link1
- removed link Link10
- removed link Link2
- removed link Link3
- removed link Link4
- removed link Link5
- removed link Link6
- removed link Link7
- removed link Link8
- removed link Link9
- added link LeftLink0, mass 1; collision box size=0.15146327406410975 0.39525510101266226 0.47646985567856914; visual box size=0.15146327406410975 0.39525510101266226 0.47646985567856914
- added link LeftLink1, mass 1; collision box size=0.08498013645436908 0.3818982218334358 0.4655114490780352; visual box size=0.08498013645436908 0.3818982218334358 0.4655114490780352
- added link LeftLink2, mass 1; collision box size=0.8671698926157774 0.5389391242916889 0.7867751310369935; visual box size=0.8671698926157774 0.5389391242916889 0.7867751310369935
- added link LeftLink3, mass 1; collision box size=0.2591761951634459 0.07496747014955585 0.7837341624427193; visual box size=0.2591761951634459 0.07496747014955585 0.7837341624427193
- added link LeftLink4, mass 1; collision box size=0.030510979749644562 0.3683483229379745 0.9461063771987192; visual box size=0.030510979749644562 0.3683483229379745 0.9461063771987192
- added link LeftLink5, mass 1; collision box size=0.10036159732585748 0.23344973215412346 0.9546716213446287; visual box size=0.10036159732585748 0.23344973215412346 0.9546716213446287
- added link LeftLink6, mass 1; collision box size=0.113253489897576 0.8862025985801928 0.43703509169499066; visual box size=0.113253489897576 0.8862025985801928 0.43703509169499066
- added link LeftLink7, mass 1; collision box size=0.3041670890698511 0.9488071195765505 0.029350538486849875; visual box size=0.3041670890698511 0.9488071195765505 0.029350538486849875
- added link RightLink0, mass 1; collision box size=0.15146327406410975 0.39525510101266226 0.47646985567856914; visual box size=0.15146327406410975 0.39525510101266226 0.47646985567856914
- added link RightLink1, mass 1; collision box size=0.08498013645436908 0.3818982218334358 0.4655114490780352; visual box size=0.08498013645436908 0.3818982218334358 0.4655114490780352
- added link RightLink2, mass 1; collision box size=0.8671698926157774 0.5389391242916889 0.7867751310369935; visual box size=0.8671698926157774 0.5389391242916889 0.7867751310369935
- added link RightLink3, mass 1; collision box size=0.2591761951634459 0.07496747014955585 0.7837341624427193; visual box size=0.2591761951634459 0.07496747014955585 0.7837341624427193
- added link RightLink4, mass 1; collision box size=0.030510979749644562 0.3683483229379745 0.9461063771987192; visual box size=0.030510979749644562 0.3683483229379745 0.9461063771987192
- added link RightLink5, mass 1; collision box size=0.10036159732585748 0.23344973215412346 0.9546716213446287; visual box size=0.10036159732585748 0.23344973215412346 0.9546716213446287
- added link RightLink6, mass 1; collision box size=0.113253489897576 0.8862025985801928 0.43703509169499066; visual box size=0.113253489897576 0.8862025985801928 0.43703509169499066
- added link RightLink7, mass 1; collision box size=0.3041670890698511 0.9488071195765505 0.029350538486849875; visual box size=0.3041670890698511 0.9488071195765505 0.029350538486849875
Joints:
- removed joint Link0_Link1
- removed joint Link1_Link2
- removed joint Link2_Link3
- removed joint Link3_Link4
- removed joint Link4_Link5
- removed joint Link5_Link6
- removed joint Link6_Link7
- removed joint Link7_Link8
- removed joint Link8_Link9
- removed joint Link9_Link10
- added joint LeftLink0_LeftLink1: type revolute, parent LeftLink0, child eftLink1, origin xyz=0 0.5 0 rpy=0 0 0, axis 1 1 0, limit lower=-3.14159 upper=3.14159 effort=0.0 velocity=0.0
- added joint LeftLink1_LeftLink2: type revolute, parent LeftLink1, child eftLink2, origin xyz=0 0.5 0 rpy=0 0 0, axis 1 1 0, limit lower=-3.14159 upper=3.14159 effort=0.0 velocity=0.0
- added joint LeftLink2_LeftLink3: type revolute, parent LeftLink2, child eftLink3, origin xyz=0 0.5 0 rpy=0 0 0, axis 1 1 0, limit lower=-3.14159 upper=3.14159 effort=0.0 velocity=0.0
- added joint LeftLink3_LeftLink4: type revolute, parent LeftLink3, child eftLink4, origin xyz=0 0.5 0 rpy=0 0 0, axis 1 1 0, limit lower=-3.14159 upper=3.14159 effort=0.0 velocity=0.0
- added joint LeftLink4_LeftLink5: type revolute, parent LeftLink4, child eftLink5, origin xyz=0 0.5 0 rpy=0 0 0, axis 1 1 0, limit lower=-3.14159 upper=3.14159 effort=0.0 velocity=0.0
- added joint LeftLink5_LeftLink6: type revolute, parent LeftLink5, child eftLink6, origin xyz=0 0.5 0 rpy=0 0 0, axis 1 1 0, limit lower=-3.14159 upper=3.14159 effort=0.0 velocity=0.0
- added joint LeftLink6_LeftLink7: type revolute, parent LeftLink6, child eftLink7, origin xyz=0 0.5 0 rpy=0 0 0, axis 1 1 0, limit lower=-3.14159 upper=3.14159 effort=0.0 velocity=0.0
- added joint RightLink0_RightLink1: type revolute, parent RightLink0, child ightLink1, origin xyz=0 0.5 0 rpy=0 0 0, axis 1 1 0, limit lower=-3.14159 upper=3.14159 effort=0.0 velocity=0.0
- added joint RightLink1_RightLink2: type revolute, parent RightLink1, child ightLink2, origin xyz=0 0.5 0 rpy=0 0 0, axis 1 1 0, limit lower=-3.14159 upper=3.14159 effort=0.0 velocity=0.0
- added joint RightLink2_RightLink3: type revolute, parent RightLink2, child ightLink3, origin xyz=0 0.5 0 rpy=0 0 0, axis 1 1 0, limit lower=-3.14159 upper=3.14159 effort=0.0 velocity=0.0
- added joint RightLink3_RightLink4: type revolute, parent RightLink3, child ightLink4, origin xyz=0 0.5 0 rpy=0 0 0, axis 1 1 0, limit lower=-3.14159 upper=3.14159 effort=0.0 velocity=0.0
- added joint RightLink4_RightLink5: type revolute, parent RightLink4, child ightLink5, origin xyz=0 0.5 0 rpy=0 0 0, axis 1 1 0, limit lower=-3.14159 upper=3.14159 effort=0.0 velocity=0.0
- added joint RightLink5_RightLink6: type revolute, parent RightLink5, child ightLink6, origin xyz=0 0.5 0 rpy=0 0 0, axis 1 1 0, limit lower=-3.14159 upper=3.14159 effort=0.0 velocity=0.0
- added joint RightLink6_RightLink7: type revolute, parent RightLink6, child ightLink7, origin xyz=0 0.5 0 rpy=0 0 0, axis 1 1 0, limit lower=-3.14159 upper=3.14159 effort=0.0 velocity=0.0
- joint Torso_Link0: origin xyz=0 2.25 0.5 rpy=0 0 0 -> xyz=0 2.25 4.75 rpy=0 0 0

Commit message: etc

File: body.urdf (robot description, URDF)
Before this commit: robot robot, 17 links, 15 joints
Links:
- added link LeftLink10, mass 1; collision box size=0.8399245111497322 0.795341266304772 0.8537172142377708; visual box size=0.8399245111497322 0.795341266304772 0.8537172142377708
- added link LeftLink8, mass 1; collision box size=0.9767276982178947 0.24441857916391063 0.46931749300308645; visual box size=0.9767276982178947 0.24441857916391063 0.46931749300308645
- added link LeftLink9, mass 1; collision box size=0.4537301571499689 0.8898275867981407 0.26133831684566144; visual box size=0.4537301571499689 0.8898275867981407 0.26133831684566144
- added link RightLink10, mass 1; collision box size=0.8399245111497322 0.795341266304772 0.8537172142377708; visual box size=0.8399245111497322 0.795341266304772 0.8537172142377708
- added link RightLink8, mass 1; collision box size=0.9767276982178947 0.24441857916391063 0.46931749300308645; visual box size=0.9767276982178947 0.24441857916391063 0.46931749300308645
- added link RightLink9, mass 1; collision box size=0.4537301571499689 0.8898275867981407 0.26133831684566144; visual box size=0.4537301571499689 0.8898275867981407 0.26133831684566144
- link LeftLink0: geometry collision box size=0.6265015869215932 0.8759043605662777 0.39644034294134667; visual box size=0.6265015869215932 0.8759043605662777 0.39644034294134667
- link LeftLink1: geometry collision box size=0.07095063344550778 0.28568632581745146 0.3089096438260416; visual box size=0.07095063344550778 0.28568632581745146 0.3089096438260416
- link LeftLink2: geometry collision box size=0.42799367033491564 0.7909681260355276 0.6868890911453087; visual box size=0.42799367033491564 0.7909681260355276 0.6868890911453087
- link LeftLink3: geometry collision box size=0.10932471492117779 0.4741183786606654 0.7530045053944229; visual box size=0.10932471492117779 0.4741183786606654 0.7530045053944229
- link LeftLink4: geometry collision box size=0.5522475167125668 0.7306202779339102 0.790914681293578; visual box size=0.5522475167125668 0.7306202779339102 0.790914681293578
- link LeftLink5: geometry collision box size=0.2823153076276218 0.14874249355777802 0.7816821123396723; visual box size=0.2823153076276218 0.14874249355777802 0.7816821123396723
- link LeftLink6: geometry collision box size=0.022083856030610916 0.5270431900388541 0.556574934355055; visual box size=0.022083856030610916 0.5270431900388541 0.556574934355055
- link LeftLink7: geometry collision box size=0.640213295925364 0.8243262019551382 0.7849873388386022; visual box size=0.640213295925364 0.8243262019551382 0.7849873388386022
- link RightLink0: geometry collision box size=0.6265015869215932 0.8759043605662777 0.39644034294134667; visual box size=0.6265015869215932 0.8759043605662777 0.39644034294134667
- link RightLink1: geometry collision box size=0.07095063344550778 0.28568632581745146 0.3089096438260416; visual box size=0.07095063344550778 0.28568632581745146 0.3089096438260416
- link RightLink2: geometry collision box size=0.42799367033491564 0.7909681260355276 0.6868890911453087; visual box size=0.42799367033491564 0.7909681260355276 0.6868890911453087
- link RightLink3: geometry collision box size=0.10932471492117779 0.4741183786606654 0.7530045053944229; visual box size=0.10932471492117779 0.4741183786606654 0.7530045053944229
- link RightLink4: geometry collision box size=0.5522475167125668 0.7306202779339102 0.790914681293578; visual box size=0.5522475167125668 0.7306202779339102 0.790914681293578
- link RightLink5: geometry collision box size=0.2823153076276218 0.14874249355777802 0.7816821123396723; visual box size=0.2823153076276218 0.14874249355777802 0.7816821123396723
- link RightLink6: geometry collision box size=0.022083856030610916 0.5270431900388541 0.556574934355055; visual box size=0.022083856030610916 0.5270431900388541 0.556574934355055
- link RightLink7: geometry collision box size=0.640213295925364 0.8243262019551382 0.7849873388386022; visual box size=0.640213295925364 0.8243262019551382 0.7849873388386022
Joints:
- added joint LeftLink7_LeftLink8: type revolute, parent LeftLink7, child eftLink8, origin xyz=0 0.5 0 rpy=0 0 0, axis 1 1 0, limit lower=-3.14159 upper=3.14159 effort=0.0 velocity=0.0
- added joint LeftLink8_LeftLink9: type revolute, parent LeftLink8, child eftLink9, origin xyz=0 0.5 0 rpy=0 0 0, axis 1 1 0, limit lower=-3.14159 upper=3.14159 effort=0.0 velocity=0.0
- added joint LeftLink9_LeftLink10: type revolute, parent LeftLink9, child eftLink10, origin xyz=0 0.5 0 rpy=0 0 0, axis 1 1 0, limit lower=-3.14159 upper=3.14159 effort=0.0 velocity=0.0
- added joint RightLink7_RightLink8: type revolute, parent RightLink7, child ightLink8, origin xyz=0 0.5 0 rpy=0 0 0, axis 1 1 0, limit lower=-3.14159 upper=3.14159 effort=0.0 velocity=0.0
- added joint RightLink8_RightLink9: type revolute, parent RightLink8, child ightLink9, origin xyz=0 0.5 0 rpy=0 0 0, axis 1 1 0, limit lower=-3.14159 upper=3.14159 effort=0.0 velocity=0.0
- added joint RightLink9_RightLink10: type revolute, parent RightLink9, child ightLink10, origin xyz=0 0.5 0 rpy=0 0 0, axis 1 1 0, limit lower=-3.14159 upper=3.14159 effort=0.0 velocity=0.0

Commit message: post OH

File: body.urdf (robot description, URDF)
Before this commit: robot robot, 23 links, 21 joints
Links:
- link LeftLink0: geometry collision box size=0.6758111505934802 0.4043326982704415 0.5007347387398641; visual box size=0.6758111505934802 0.4043326982704415 0.5007347387398641
- link LeftLink1: geometry collision box size=0.7657926160734788 0.13184358670242757 0.12131709457562234; visual box size=0.7657926160734788 0.13184358670242757 0.12131709457562234
- link LeftLink10: geometry collision box size=0.2868838881852843 0.026872955395925713 0.08534544779641673; visual box size=0.2868838881852843 0.026872955395925713 0.08534544779641673
- link LeftLink2: geometry collision box size=0.31086306249713036 0.5089521486547077 0.49818833740184665; visual box size=0.31086306249713036 0.5089521486547077 0.49818833740184665
- link LeftLink3: geometry collision box size=0.046745081059601845 0.34970774215511136 0.9361783244530244; visual box size=0.046745081059601845 0.34970774215511136 0.9361783244530244
- link LeftLink4: geometry collision box size=0.813649496243857 0.9746350589125302 0.7004705959624002; visual box size=0.813649496243857 0.9746350589125302 0.7004705959624002
- link LeftLink5: geometry collision box size=0.7658875800092235 0.9753861114157342 0.16662103494302116; visual box size=0.7658875800092235 0.9753861114157342 0.16662103494302116
- link LeftLink6: geometry collision box size=0.8800184017737652 0.9812178753036117 0.23860746250271714; visual box size=0.8800184017737652 0.9812178753036117 0.23860746250271714
- link LeftLink7: geometry collision box size=0.14124226965458497 0.8637794823920913 0.5937427616707075; visual box size=0.14124226965458497 0.8637794823920913 0.5937427616707075
- link LeftLink8: geometry collision box size=0.8200447468242871 0.711412200169552 0.7961369119826208; visual box size=0.8200447468242871 0.711412200169552 0.7961369119826208
- link LeftLink9: geometry collision box size=0.18301809495628463 0.4364497830236306 0.872697126162834; visual box size=0.18301809495628463 0.4364497830236306 0.872697126162834
- link RightLink0: geometry collision box size=0.6758111505934802 0.4043326982704415 0.5007347387398641; visual box size=0.6758111505934802 0.4043326982704415 0.5007347387398641
- link RightLink1: geometry collision box size=0.7657926160734788 0.13184358670242757 0.12131709457562234; visual box size=0.7657926160734788 0.13184358670242757 0.12131709457562234
- link RightLink10: geometry collision box size=0.2868838881852843 0.026872955395925713 0.08534544779641673; visual box size=0.2868838881852843 0.026872955395925713 0.08534544779641673
- link RightLink2: geometry collision box size=0.31086306249713036 0.5089521486547077 0.49818833740184665; visual box size=0.31086306249713036 0.5089521486547077 0.49818833740184665
- link RightLink3: geometry collision box size=0.046745081059601845 0.34970774215511136 0.9361783244530244; visual box size=0.046745081059601845 0.34970774215511136 0.9361783244530244
- link RightLink4: geometry collision box size=0.813649496243857 0.9746350589125302 0.7004705959624002; visual box size=0.813649496243857 0.9746350589125302 0.7004705959624002
- link RightLink5: geometry collision box size=0.7658875800092235 0.9753861114157342 0.16662103494302116; visual box size=0.7658875800092235 0.9753861114157342 0.16662103494302116
- link RightLink6: geometry collision box size=0.8800184017737652 0.9812178753036117 0.23860746250271714; visual box size=0.8800184017737652 0.9812178753036117 0.23860746250271714
- link RightLink7: geometry collision box size=0.14124226965458497 0.8637794823920913 0.5937427616707075; visual box size=0.14124226965458497 0.8637794823920913 0.5937427616707075
- link RightLink8: geometry collision box size=0.8200447468242871 0.711412200169552 0.7961369119826208; visual box size=0.8200447468242871 0.711412200169552 0.7961369119826208
- link RightLink9: geometry collision box size=0.18301809495628463 0.4364497830236306 0.872697126162834; visual box size=0.18301809495628463 0.4364497830236306 0.872697126162834
