Commit message: debugging! made it to Brain :)

File: body.urdf (robot description, URDF)
Before this commit: robot robot, 23 links, 21 joints
Links:
- removed link LeftLink0
- removed link LeftLink1
- removed link LeftLink10
- removed link LeftLink2
- removed link LeftLink3
- removed link LeftLink4
- removed link LeftLink5
- removed link LeftLink6
- removed link LeftLink7
- removed link LeftLink8
- removed link LeftLink9
- removed link RightLink0
- removed link RightLink1
- removed link RightLink10
- removed link RightLink2
- removed link RightLink3
- removed link RightLink4
- removed link RightLink5
- removed link RightLink6
- removed link RightLink7
- removed link RightLink8
- removed link RightLink9
- added link 0Link0, mass 1; collision box size=0.20010266365867357 0.9291371170856926 0.7359910875978013; visual box size=0.20010266365867357 0.9291371170856926 0.7359910875978013
- added link 0Link1, mass 1; collision box size=0.5828165681255993 0.5708586808134645 0.4195037096566687; visual box size=0.5828165681255993 0.5708586808134645 0.4195037096566687
- added link 0Link2, mass 1; collision box size=0.8037427006842252 0.11745688722093195 0.9787831497828227; visual box size=0.8037427006842252 0.11745688722093195 0.9787831497828227
- added link 0Link3, mass 1; collision box size=0.3086148087595235 0.5193943010074328 0.19959053458619036; visual box size=0.3086148087595235 0.5193943010074328 0.19959053458619036
- added link 0Link4, mass 1; collision box size=0.14447560603719267 0.09283820819321076 0.0768440050261261; visual box size=0.14447560603719267 0.09283820819321076 0.0768440050261261
- added link 0Link5, mass 1; collision box size=0.0008357696293319616 0.5613756994836014 0.3840253340496066; visual box size=0.0008357696293319616 0.5613756994836014 0.3840253340496066
- added link 0Link6, mass 1; collision box size=0.5186837739657103 0.3172208746309516 0.14946519051584795; visual box size=0.5186837739657103 0.3172208746309516 0.14946519051584795
- added link 0Link7, mass 1; collision box size=0.7895894000831188 0.5571414659827968 0.009611750734853763; visual box size=0.7895894000831188 0.5571414659827968 0.009611750734853763
- added link 0Link8, mass 1; collision box size=0.7012879992591696 0.03476282227046146 0.9390501510604254; visual box size=0.7012879992591696 0.03476282227046146 0.9390501510604254
- added link 1Link0, mass 1; collision box size=0.10412649429060117 0.06342321466937706 0.4641702847589676; visual box size=0.10412649429060117 0.06342321466937706 0.4641702847589676
- added link 1Link1, mass 1; collision box size=0.7858016609862026 0.36661266038410734 0.7471916720325523; visual box size=0.7858016609862026 0.36661266038410734 0.7471916720325523
- added link 1Link2, mass 1; collision box size=0.7463143255024531 0.7942866664725303 0.7176533852122505; visual box size=0.7463143255024531 0.7942866664725303 0.7176533852122505
- added link 1Link3, mass 1; collision box size=0.44297383347876684 0.33150154421585487 0.6702531430338968; visual box size=0.44297383347876684 0.33150154421585487 0.6702531430338968
- added link 1Link4, mass 1; collision box size=0.32634096443153027 0.9916698914296631 0.3690557462437155; visual box size=0.32634096443153027 0.9916698914296631 0.3690557462437155
- added link 1Link5, mass 1; collision box size=0.5221352057735851 0.6315859566257429 0.4526976942497306; visual box size=0.5221352057735851 0.6315859566257429 0.4526976942497306
- added link 1Link6, mass 1; collision box size=0.4417824576481214 0.8892862547719805 0.016391501503053796; visual box size=0.4417824576481214 0.8892862547719805 0.016391501503053796
- added link 1Link7, mass 1; collision box size=0.2732423978472862 0.4434943510672099 0.22497329814931188; visual box size=0.2732423978472862 0.4434943510672099 0.22497329814931188
- added link 2Link0, mass 1; collision box size=0.6874889574346795 0.9524764586550398 0.7566206165096957; visual box size=0.6874889574346795 0.9524764586550398 0.7566206165096957
- added link 2Link1, mass 1; collision box size=0.6567263570202095 0.12885615256648741 0.2405124423243934; visual box size=0.6567263570202095 0.12885615256648741 0.2405124423243934
- added link 2Link2, mass 1; collision box size=0.8022284555373326 0.5622414142864378 0.8998447361274039; visual box size=0.8022284555373326 0.5622414142864378 0.8998447361274039
- added link 2Link3, mass 1; collision box size=0.766551934448767 0.3904506518570452 0.5576056381219434; visual box size=0.766551934448767 0.3904506518570452 0.5576056381219434
- added link 2Link4, mass 1; collision box size=0.8438657131464222 0.4910995890031473 0.6455316693558407; visual box size=0.8438657131464222 0.4910995890031473 0.6455316693558407
- added link 2Link5, mass 1; collision box size=0.25796765320748716 0.5994445891806551 0.3998910656823783; visual box size=0.25796765320748716 0.5994445891806551 0.3998910656823783
- added link 2Link6, mass 1; collision box size=0.9683646649549095 0.6927485141272784 0.6176216763712848; visual box size=0.9683646649549095 0.6927485141272784 0.6176216763712848
- added link 2Link7, mass 1; collision box size=0.9218775482696671 0.5143547939520373 0.08129565498113567; visual box size=0.9218775482696671 0.5143547939520373 0.08129565498113567
- added link 3Link0, mass 1; collision box size=0.0018411815100021212 0.008629913071303341 0.37249269648475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; visual box size=0.0018411815100021212 0.008629913071303341 0.37249269648475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
- added link 3Link1, mass 1; collision box size=0.29417333509063837 0.29491099908495666 0.29184952684105836; visual box size=0.29417333509063837 0.29491099908495666 0.29184952684105836
- added link 3Link2, mass 1; collision box size=0.5198793355035409 0.2592605389662237 0.25750502231692374; visual box size=0.5198793355035409 0.2592605389662237 0.25750502231692374
- added link 3Link3, mass 1; collision box size=0.43342144640656777 0.07383729450999055 0.15688291988980063; visual box size=0.43342144640656777 0.07383729450999055 0.15688291988980063
- added link 3Link4, mass 1; collision box size=0.7081942144262235 0.09648842840223992 0.1410300490977845; visual box size=0.7081942144262235 0.09648842840223992 0.1410300490977845
- added link 3Link5, mass 1; collision box size=0.14067424446927723 0.14085057622353014 0.44582429389553413; visual box size=0.14067424446927723 0.14085057622353014 0.44582429389553413
- added link 3Link6, mass 1; collision box size=0.49497732862530563 0.5543247331569873 0.3848607238147076; visual box size=0.49497732862530563 0.5543247331569873 0.3848607238147076
- added link 3Link7, mass 1; collision box size=0.7193089774075668 0.21843721677434114 0.8831432121322184; visual box size=0.7193089774075668 0.21843721677434114 0.8831432121322184
- added link 3Link8, mass 1; collision box size=0.7903399976191366 0.869817680151397 0.11284248788756068; visual box size=0.7903399976191366 0.869817680151397 0.11284248788756068
- added link 3Link9, mass 1; collision box size=0.7857524371551784 0.17076342806809053 0.5586975971228596; visual box size=0.7857524371551784 0.17076342806809053 0.5586975971228596
Joints:
- removed joint LeftLink0_LeftLink1
- removed joint LeftLink1_LeftLink2
- removed joint LeftLink2_LeftLink3
- removed joint LeftLink3_LeftLink4
- removed joint LeftLink4_LeftLink5
- removed joint LeftLink5_LeftLink6
- removed joint LeftLink6_LeftLink7
- removed joint LeftLink7_LeftLink8
- removed joint LeftLink8_LeftLink9
- removed joint LeftLink9_LeftLink10
- removed joint RightLink0_RightLink1
- removed joint RightLink1_RightLink2
- removed joint RightLink2_RightLink3
- removed joint RightLink3_RightLink4
- removed joint RightLink4_RightLink5
- removed joint RightLink5_RightLink6
- removed joint RightLink6_RightLink7
- removed joint RightLink7_RightLink8
- removed joint RightLink8_RightLink9
- removed joint RightLink9_RightLink10
- removed joint Torso_Link0
- added joint 0Link0_0Link1: type revolute, parent 0Link0, child 0Link1, origin xyz=0 0.5 0 rpy=0 0 0, axis 1 1 0, limit lower=-3.14159 upper=3.14159 effort=0.0 velocity=0.0
- added joint 0Link1_0Link2: type revolute, parent 0Link1, child 0Link2, origin xyz=0 0.5 0 rpy=0 0 0, axis 1 1 0, limit lower=-3.14159 upper=3.14159 effort=0.0 velocity=0.0
- added joint 0Link2_0Link3: type revolute, parent 0Link2, child 0Link3, origin xyz=0 0.5 0 rpy=0 0 0, axis 1 1 0, limit lower=-3.14159 upper=3.14159 effort=0.0 velocity=0.0
- added joint 0Link3_0Link4: type revolute, parent 0Link3, child 0Link4, origin xyz=0 0.5 0 rpy=0 0 0, axis 1 1 0, limit lower=-3.14159 upper=3.14159 effort=0.0 velocity=0.0
- added joint 0Link4_0Link5: type revolute, parent 0Link4, child 0Link5, origin xyz=0 0.5 0 rpy=0 0 0, axis 1 1 0, limit lower=-3.14159 upper=3.14159 effort=0.0 velocity=0.0
- added joint 0Link5_0Link6: type revolute, parent 0Link5, child 0Link6, origin xyz=0 0.5 0 rpy=0 0 0, axis 1 1 0, limit lower=-3.14159 upper=3.14159 effort=0.0 velocity=0.0
- added joint 0Link6_0Link7: type revolute, parent 0Link6, child 0Link7, origin xyz=0 0.5 0 rpy=0 0 0, axis 1 1 0, limit lower=-3.14159 upper=3.14159 effort=0.0 velocity=0.0
- added joint 0Link7_0Link8: type revolute, parent 0Link7, child 0Link8, origin xyz=0 0.5 0 rpy=0 0 0, axis 1 1 0, limit lower=-3.14159 upper=3.14159 effort=0.0 velocity=0.0
- added joint 1Link0_1Link1: type revolute, parent 1Link0, child 1Link1, origin xyz=0 0.5 0 rpy=0 0 0, axis 1 1 0, limit lower=-3.14159 upper=3.14159 effort=0.0 velocity=0.0
- added joint 1Link1_1Link2: type revolute, parent 1Link1, child 1Link2, origin xyz=0 0.5 0 rpy=0 0 0, axis 1 1 0, limit lower=-3.14159 upper=3.14159 effort=0.0 velocity=0.0
- added joint 1Link2_1Link3: type revolute, parent 1Link2, child 1Link3, origin xyz=0 0.5 0 rpy=0 0 0, axis 1 1 0, limit lower=-3.14159 upper=3.14159 effort=0.0 velocity=0.0
- added joint 1Link3_1Link4: type revolute, parent 1Link3, child 1Link4, origin xyz=0 0.5 0 rpy=0 0 0, axis 1 1 0, limit lower=-3.14159 upper=3.14159 effort=0.0 velocity=0.0
- added joint 1Link4_1Link5: type revolute, parent 1Link4, child 1Link5, origin xyz=0 0.5 0 rpy=0 0 0, axis 1 1 0, limit lower=-3.14159 upper=3.14159 effort=0.0 velocity=0.0
- added joint 1Link5_1Link6: type revolute, parent 1Link5, child 1Link6, origin xyz=0 0.5 0 rpy=0 0 0, axis 1 1 0, limit lower=-3.14159 upper=3.14159 effort=0.0 velocity=0.0
- added joint 1Link6_1Link7: type revolute, parent 1Link6, child 1Link7, origin xyz=0 0.5 0 rpy=0 0 0, axis 1 1 0, limit lower=-3.14159 upper=3.14159 effort=0.0 velocity=0.0
- added joint 2Link0_2Link1: type revolute, parent 2Link0, child 2Link1, origin xyz=0 0.5 0 rpy=0 0 0, axis 1 1 0, limit lower=-3.14159 upper=3.14159 effort=0.0 velocity=0.0
- added joint 2Link1_2Link2: type revolute, parent 2Link1, child 2Link2, origin xyz=0 0.5 0 rpy=0 0 0, axis 1 1 0, limit lower=-3.14159 upper=3.14159 effort=0.0 velocity=0.0
- added joint 2Link2_2Link3: type revolute, parent 2Link2, child 2Link3, origin xyz=0 0.5 0 rpy=0 0 0, axis 1 1 0, limit lower=-3.14159 upper=3.14159 effort=0.0 velocity=0.0
- added joint 2Link3_2Link4: type revolute, parent 2Link3, child 2Link4, origin xyz=0 0.5 0 rpy=0 0 0, axis 1 1 0, limit lower=-3.14159 upper=3.14159 effort=0.0 velocity=0.0
- added joint 2Link4_2Link5: type revolute, parent 2Link4, child 2Link5, origin xyz=0 0.5 0 rpy=0 0 0, axis 1 1 0, limit lower=-3.14159 upper=3.14159 effort=0.0 velocity=0.0
- added joint 2Link5_2Link6: type revolute, parent 2Link5, child 2Link6, origin xyz=0 0.5 0 rpy=0 0 0, axis 1 1 0, limit lower=-3.14159 upper=3.14159 effort=0.0 velocity=0.0
- added joint 2Link6_2Link7: type revolute, parent 2Link6, child 2Link7, origin xyz=0 0.5 0 rpy=0 0 0, axis 1 1 0, limit lower=-3.14159 upper=3.14159 effort=0.0 velocity=0.0
- added joint 3Link0_3Link1: type revolute, parent 3Link0, child 3Link1, origin xyz=0 0.5 0 rpy=0 0 0, axis 1 1 0, limit lower=-3.14159 upper=3.14159 effort=0.0 velocity=0.0
- added joint 3Link1_3Link2: type revolute, parent 3Link1, child 3Link2, origin xyz=0 0.5 0 rpy=0 0 0, axis 1 1 0, limit lower=-3.14159 upper=3.14159 effort=0.0 velocity=0.0
- added joint 3Link2_3Link3: type revolute, parent 3Link2, child 3Link3, origin xyz=0 0.5 0 rpy=0 0 0, axis 1 1 0, limit lower=-3.14159 upper=3.14159 effort=0.0 velocity=0.0
- added joint 3Link3_3Link4: type revolute, parent 3Link3, child 3Link4, origin xyz=0 0.5 0 rpy=0 0 0, axis 1 1 0, limit lower=-3.14159 upper=3.14159 effort=0.0 velocity=0.0
- added joint 3Link4_3Link5: type revolute, parent 3Link4, child 3Link5, origin xyz=0 0.5 0 rpy=0 0 0, axis 1 1 0, limit lower=-3.14159 upper=3.14159 effort=0.0 velocity=0.0
- added joint 3Link5_3Link6: type revolute, parent 3Link5, child 3Link6, origin xyz=0 0.5 0 rpy=0 0 0, axis 1 1 0, limit lower=-3.14159 upper=3.14159 effort=0.0 velocity=0.0
- added joint 3Link6_3Link7: type revolute, parent 3Link6, child 3Link7, origin xyz=0 0.5 0 rpy=0 0 0, axis 1 1 0, limit lower=-3.14159 upper=3.14159 effort=0.0 velocity=0.0
- added joint 3Link7_3Link8: type revolute, parent 3Link7, child 3Link8, origin xyz=0 0.5 0 rpy=0 0 0, axis 1 1 0, limit lower=-3.14159 upper=3.14159 effort=0.0 velocity=0.0
- added joint 3Link8_3Link9: type revolute, parent 3Link8, child 3Link9, origin xyz=0 0.5 0 rpy=0 0 0, axis 1 1 0, limit lower=-3.14159 upper=3.14159 effort=0.0 velocity=0.0
- added joint Torso_Base0: type revolute, parent Torso, child Base0, origin xyz=0.0 2.0 9.0 rpy=0 0 0, axis 1 1 0, limit lower=-3.14159 upper=3.14159 effort=0.0 velocity=0.0
- added joint Torso_Base1: type revolute, parent Torso, child Base1, origin xyz=-1.0 2.0 10.0 rpy=0 0 0, axis 1 1 0, limit lower=-3.14159 upper=3.14159 effort=0.0 velocity=0.0
- added joint Torso_Base2: type revolute, parent Torso, child Base2, origin xyz=0.0 2.0 10.0 rpy=0 0 0, axis 1 1 0, limit lower=-3.14159 upper=3.14159 effort=0.0 velocity=0.0
- added joint Torso_Base3: type revolute, parent Torso, child Base3, origin xyz=0.0 2.0 10.0 rpy=0 0 0, axis 1 1 0, limit lower=-3.14159 upper=3.14159 effort=0.0 velocity=0.0

Commit message: getting close

File: body.urdf (robot description, URDF)
Before this commit: robot robot, 26 links, 25 joints
Links:
- removed link 2Link0
- removed link 2Link1
- removed link 2Link2
- removed link 2Link3
- removed link 2Link4
- removed link 2Link5
- removed link 2Link6
- removed link 2Link7
- removed link 2Link8
- added link 1Link8, mass 1; collision box size=0.362781589325174 0.12685344731103398 0.9530023420977044; visual box size=0.362781589325174 0.12685344731103398 0.9530023420977044
- link 0Link0: geometry collision box size=0.9480638686895049 0.636282397920891 0.42506167459574795; visual box size=0.9480638686895049 0.636282397920891 0.42506167459574795
- link 0Link1: geometry collision box size=0.3797322411657893 0.6054803343662202 0.8407664047518844; visual box size=0.3797322411657893 0.6054803343662202 0.8407664047518844
- link 0Link2: geometry collision box size=0.6459821155129104 0.8441508811626253 0.8188966894262356; visual box size=0.6459821155129104 0.8441508811626253 0.8188966894262356
- link 0Link3: geometry collision box size=0.27685609452121007 0.4413660360604196 0.45120860655481754; visual box size=0.27685609452121007 0.4413660360604196 0.45120860655481754
- link 0Link4: geometry collision box size=0.35096750710820623 0.6355437494434677 0.4609801012662854; visual box size=0.35096750710820623 0.6355437494434677 0.4609801012662854
- link 0Link5: geometry collision box size=0.9113618709793779 0.43774669289795887 0.7335713844120337; visual box size=0.9113618709793779 0.43774669289795887 0.7335713844120337
- link 0Link6: geometry collision box size=0.32813600536717014 0.1709607976447245 0.11890367471990038; visual box size=0.32813600536717014 0.1709607976447245 0.11890367471990038
- link 0Link7: geometry collision box size=0.7316370425043239 0.36082877738745145 0.4235384562633615; visual box size=0.7316370425043239 0.36082877738745145 0.4235384562633615
- link 1Link0: geometry collision box size=0.36712876177116327 0.0028225760746171114 0.300327395773627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; visual box size=0.36712876177116327 0.0028225760746171114 0.300327395773627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
- link 1Link1: geometry collision box size=0.5929539866873461 0.6107411805855367 0.8222488127026641; visual box size=0.5929539866873461 0.6107411805855367 0.8222488127026641
- link 1Link2: geometry collision box size=0.2188439677605808 0.8321784692734122 0.07330264442094914; visual box size=0.2188439677605808 0.8321784692734122 0.07330264442094914
- link 1Link3: geometry collision box size=0.6461900489847068 0.2453532192580522 0.10103472420465387; visual box size=0.6461900489847068 0.2453532192580522 0.10103472420465387
- link 1Link4: geometry collision box size=0.7058528961142295 0.8915105857362684 0.5170263872062076; visual box size=0.7058528961142295 0.8915105857362684 0.5170263872062076
- link 1Link5: geometry collision box size=0.7964751957640877 0.7858987007333765 0.9029859333130976; visual box size=0.7964751957640877 0.7858987007333765 0.9029859333130976
- link 1Link6: geometry collision box size=0.14753973558389977 0.7088712703000294 0.6055103786966701; visual box size=0.14753973558389977 0.7088712703000294 0.6055103786966701
- link 1Link7: geometry collision box size=0.6559880385392101 0.8334679225408884 0.7662808190514165; visual box size=0.6559880385392101 0.8334679225408884 0.7662808190514165
Joints:
- removed joint 2Link0_2Link1
- removed joint 2Link1_2Link2
- removed joint 2Link2_2Link3
- removed joint 2Link3_2Link4
- removed joint 2Link4_2Link5
- removed joint 2Link5_2Link6
- removed joint 2Link6_2Link7
- removed joint 2Link7_2Link8
- removed joint Torso_Base2
- added joint 1Link7_1Link8: type revolute, parent 1Link7, child 1Link8, origin xyz=-0.5 0 0 rpy=0 0 0, axis 1 1 0, limit lower=-3.14159 upper=3.14159 effort=0.0 velocity=0.0
- joint 0Link0_0Link1: origin xyz=0 0.5 0 rpy=0 0 0 -> xyz=0 0 -0.5 rpy=0 0 0
- joint 0Link1_0Link2: origin xyz=0 0.5 0 rpy=0 0 0 -> xyz=0 0 -0.5 rpy=0 0 0
- joint 0Link2_0Link3: origin xyz=0 0.5 0 rpy=0 0 0 -> xyz=0 0 -0.5 rpy=0 0 0
- joint 0Link3_0Link4: origin xyz=0 0.5 0 rpy=0 0 0 -> xyz=0 0 -0.5 rpy=0 0 0
- joint 0Link4_0Link5: origin xyz=0 0.5 0 rpy=0 0 0 -> xyz=0 0 -0.5 rpy=0 0 0
- joint 0Link5_0Link6: origin xyz=0 0.5 0 rpy=0 0 0 -> xyz=0 0 -0.5 rpy=0 0 0
- joint 0Link6_0Link7: origin xyz=0 0.5 0 rpy=0 0 0 -> xyz=0 0 -0.5 rpy=0 0 0
- joint 1Link0_1Link1: origin xyz=0 0.5 0 rpy=0 0 0 -> xyz=-0.5 0 0 rpy=0 0 0
- joint 1Link1_1Link2: origin xyz=0 0.5 0 rpy=0 0 0 -> xyz=-0.5 0 0 rpy=0 0 0
- joint 1Link2_1Link3: origin xyz=0 0.5 0 rpy=0 0 0 -> xyz=-0.5 0 0 rpy=0 0 0
- joint 1Link3_1Link4: origin xyz=0 0.5 0 rpy=0 0 0 -> xyz=-0.5 0 0 rpy=0 0 0
- joint 1Link4_1Link5: origin xyz=0 0.5 0 rpy=0 0 0 -> xyz=-0.5 0 0 rpy=0 0 0
- joint 1Link5_1Link6: origin xyz=0 0.5 0 rpy=0 0 0 -> xyz=-0.5 0 0 rpy=0 0 0
- joint 1Link6_1Link7: origin xyz=0 0.5 0 rpy=0 0 0 -> xyz=-0.5 0 0 rpy=0 0 0
- joint Torso_Base0: origin xyz=0.0 2.0 9.0 rpy=0 0 0 -> xyz=0.0 2.0 9.5 rpy=0 0 0
- joint Torso_Base1: origin xyz=-1.0 2.0 10.0 rpy=0 0 0 -> xyz=-0.5 2.0 10.0 rpy=0 0 0
