Commit message: pretty good.

File: body.urdf (robot description, URDF)
Before this commit: robot robot, 18 links, 17 joints
Links:
- added link 0Link10, mass 1; collision box size=0.6191823439026002 0.667080170332481 0.22498098074472073; visual box size=0.6191823439026002 0.667080170332481 0.22498098074472073
- added link 0Link8, mass 1; collision box size=0.873691123456535 0.5096174692002986 0.018686218059421056; visual box size=0.873691123456535 0.5096174692002986 0.018686218059421056
- added link 0Link9, mass 1; collision box size=0.590982341047435 0.3502813079398055 0.8032084431791727; visual box size=0.590982341047435 0.3502813079398055 0.8032084431791727
- added link 2Link0, mass 1; collision box size=0.7163260318145707 0.23743605641655674 0.37603213612546005; visual box size=0.7163260318145707 0.23743605641655674 0.37603213612546005
- added link 2Link1, mass 1; collision box size=0.31497512894389956 0.21546183189268664 0.25615411716254743; visual box size=0.31497512894389956 0.21546183189268664 0.25615411716254743
- added link 2Link2, mass 1; collision box size=0.0969133758589813 0.8030595564825719 0.46117214033594045; visual box size=0.0969133758589813 0.8030595564825719 0.46117214033594045
- added link 2Link3, mass 1; collision box size=0.970505750933635 0.9943114946299643 0.9572085962570475; visual box size=0.970505750933635 0.9943114946299643 0.9572085962570475
- added link 2Link4, mass 1; collision box size=0.9175726791038579 0.44623795133237754 0.39465706137801493; visual box size=0.9175726791038579 0.44623795133237754 0.39465706137801493
- added link 2Link5, mass 1; collision box size=0.11163526398752621 0.4101598799602384 0.21583918450935413; visual box size=0.11163526398752621 0.4101598799602384 0.21583918450935413
- added link 2Link6, mass 1; collision box size=0.14364296345296756 0.5576005234069553 0.7683737563212097; visual box size=0.14364296345296756 0.5576005234069553 0.7683737563212097
- added link 2Link7, mass 1; collision box size=0.010266039971264629 0.8364999344097903 0.37967285571128406; visual box size=0.010266039971264629 0.8364999344097903 0.37967285571128406
- added link 3Link0, mass 1; collision box size=0.1521129336835907 0.22507178082394041 0.30195656968040796; visual box size=0.1521129336835907 0.22507178082394041 0.30195656968040796
- added link 3Link1, mass 1; collision box size=0.024182962292916277 0.5702598175441372 0.15368803641576; visual box size=0.024182962292916277 0.5702598175441372 0.15368803641576
- added link 3Link2, mass 1; collision box size=0.22439561463861157 0.22644479466419387 0.24540069688576283; visual box size=0.22439561463861157 0.22644479466419387 0.24540069688576283
- added link 3Link3, mass 1; collision box size=0.11984558340207274 0.22651523110083882 0.9161349568302045; visual box size=0.11984558340207274 0.22651523110083882 0.9161349568302045
- added link 3Link4, mass 1; collision box size=0.6009733328750122 0.4624676631856156 0.8217036242316126; visual box size=0.6009733328750122 0.4624676631856156 0.8217036242316126
- added link 3Link5, mass 1; collision box size=0.5256854248088688 0.3063268554703461 0.4694985584579765; visual box size=0.5256854248088688 0.3063268554703461 0.4694985584579765
- added link 3Link6, mass 1; collision box size=0.7380256593110501 0.5935413021695578 0.8368678810887397; visual box size=0.7380256593110501 0.5935413021695578 0.8368678810887397
- added link 3Link7, mass 1; collision box size=0.13154727842842173 0.8161504742513886 0.2543272689578209; visual box size=0.13154727842842173 0.8161504742513886 0.2543272689578209
- added link 3Link8, mass 1; collision box size=0.7701164076698406 0.05255300488704939 0.45687224844652374; visual box size=0.7701164076698406 0.05255300488704939 0.45687224844652374
- added link 4Link0, mass 1; collision box size=0.1294672002497994 0.23300090415444386 0.14263271723373772; visual box size=0.1294672002497994 0.23300090415444386 0.14263271723373772
- added link 4Link1, mass 1; collision box size=0.568268759659578 0.895995681714343 0.6079735186946426; visual box size=0.568268759659578 0.895995681714343 0.6079735186946426
- added link 4Link2, mass 1; collision box size=0.041730749564672376 0.26072509815471057 0.4094813311420502; visual box size=0.041730749564672376 0.26072509815471057 0.4094813311420502
- added link 4Link3, mass 1; collision box size=0.7740985766604971 0.9967819742191734 0.384111938858262; visual box size=0.7740985766604971 0.9967819742191734 0.384111938858262
- added link 4Link4, mass 1; collision box size=0.9223809048434752 0.5246591715545786 0.1550358237425551; visual box size=0.9223809048434752 0.5246591715545786 0.1550358237425551
- added link 4Link5, mass 1; collision box size=0.8591533484736429 0.4436462862086238 0.7216024465931472; visual box size=0.8591533484736429 0.4436462862086238 0.7216024465931472
- added link 4Link6, mass 1; collision box size=0.2014214782277567 0.995835509490336 0.027346958864758686; visual box size=0.2014214782277567 0.995835509490336 0.027346958864758686
- added link 4Link7, mass 1; collision box size=0.6953074049742762 0.42491573472231625 0.867877538001802; visual box size=0.6953074049742762 0.42491573472231625 0.867877538001802
- added link 4Link8, mass 1; collision box size=0.568735698751539 0.9858755388975221 0.7206810148529441; visual box size=0.568735698751539 0.9858755388975221 0.7206810148529441
- added link 4Link9, mass 1; collision box size=0.6403930786742648 0.3054183886093448 0.37266569538992256; visual box size=0.6403930786742648 0.3054183886093448 0.37266569538992256
- link 0Link0: geometry collision box size=0.11404602361424343 0.6772407137474431 0.29567618057915224; visual box size=0.11404602361424343 0.6772407137474431 0.29567618057915224
- link 0Link1: geometry collision box size=0.2145746491670889 0.06808115778987989 0.9831476687270602; visual box size=0.2145746491670889 0.06808115778987989 0.9831476687270602
- link 0Link2: geometry collision box size=0.4011531052011895 0.6785310629515737 0.7212911788018691; visual box size=0.4011531052011895 0.6785310629515737 0.7212911788018691
- link 0Link3: geometry collision box size=0.5838107784216657 0.5879220994754344 0.1486888962900319; visual box size=0.5838107784216657 0.5879220994754344 0.1486888962900319
- link 0Link4: geometry collision box size=0.4060900979974953 0.6369805859026559 0.8755781885502288; visual box size=0.4060900979974953 0.6369805859026559 0.8755781885502288
- link 0Link5: geometry collision box size=0.19046533659461806 0.35664397050647634 0.32989474907139704; visual box size=0.19046533659461806 0.35664397050647634 0.32989474907139704
- link 0Link6: geometry collision box size=0.2083110998987331 0.6595211748535085 0.32557093191864617; visual box size=0.2083110998987331 0.6595211748535085 0.32557093191864617
- link 0Link7: geometry collision box size=0.6823629396204243 0.7989662657039543 0.09806528913246415; visual box size=0.6823629396204243 0.7989662657039543 0.09806528913246415
- link 1Link0: geometry collision box size=0.23426789166955342 0.6121095263611341 0.45329547215295063; visual box size=0.23426789166955342 0.6121095263611341 0.45329547215295063
- link 1Link1: geometry collision box size=0.03400176825318646 0.7358123581499374 0.2747533303328319; visual box size=0.03400176825318646 0.7358123581499374 0.2747533303328319
- link 1Link2: geometry collision box size=0.18215496388869845 0.8234709104324351 0.46530082002587303; visual box size=0.18215496388869845 0.8234709104324351 0.46530082002587303
- link 1Link3: geometry collision box size=0.02131783992127778 0.31377035507082973 0.1657784426284249; visual box size=0.02131783992127778 0.31377035507082973 0.1657784426284249
- link 1Link4: geometry collision box size=0.6852055813096606 0.4525732343742723 0.14867134545131722; visual box size=0.6852055813096606 0.4525732343742723 0.14867134545131722
- link 1Link5: geometry collision box size=0.2698471295932705 0.0686071327132618 0.29370801931268153; visual box size=0.2698471295932705 0.0686071327132618 0.29370801931268153
- link 1Link6: geometry collision box size=0.13353596170401005 0.00994986321561786 0.42009878065087136; visual box size=0.13353596170401005 0.00994986321561786 0.42009878065087136
- link 1Link7: geometry collision box size=0.764501585168526 0.6955269677418688 0.2490662859349687; visual box size=0.764501585168526 0.6955269677418688 0.2490662859349687
- link 1Link8: geometry collision box size=0.91704020846113 0.6467301672880945 0.5543579358849322; visual box size=0.91704020846113 0.6467301672880945 0.5543579358849322
Joints:
- removed joint Torso_Base0
- removed joint Torso_Base1
- added joint 0Link7_0Link8: type revolute, parent 0Link7, child 0Link8, origin xyz=0 0 -0.5 rpy=0 0 0, axis 1 1 0, limit lower=-3.14159 upper=3.14159 effort=0.0 velocity=0.0
- added joint 0Link8_0Link9: type revolute, parent 0Link8, child 0Link9, origin xyz=0 0 -0.5 rpy=0 0 0, axis 1 1 0, limit lower=-3.14159 upper=3.14159 effort=0.0 velocity=0.0
- added joint 0Link9_0Link10: type revolute, parent 0Link9, child 0Link10, origin xyz=0 0 -0.5 rpy=0 0 0, axis 1 1 0, limit lower=-3.14159 upper=3.14159 effort=0.0 velocity=0.0
- added joint 2Link0_2Link1: type revolute, parent 2Link0, child 2Link1, origin xyz=0 0 0.5 rpy=0 0 0, axis 1 1 0, limit lower=-3.14159 upper=3.14159 effort=0.0 velocity=0.0
- added joint 2Link1_2Link2: type revolute, parent 2Link1, child 2Link2, origin xyz=0 0 0.5 rpy=0 0 0, axis 1 1 0, limit lower=-3.14159 upper=3.14159 effort=0.0 velocity=0.0
- added joint 2Link2_2Link3: type revolute, parent 2Link2, child 2Link3, origin xyz=0 0 0.5 rpy=0 0 0, axis 1 1 0, limit lower=-3.14159 upper=3.14159 effort=0.0 velocity=0.0
- added joint 2Link3_2Link4: type revolute, parent 2Link3, child 2Link4, origin xyz=0 0 0.5 rpy=0 0 0, axis 1 1 0, limit lower=-3.14159 upper=3.14159 effort=0.0 velocity=0.0
- added joint 2Link4_2Link5: type revolute, parent 2Link4, child 2Link5, origin xyz=0 0 0.5 rpy=0 0 0, axis 1 1 0, limit lower=-3.14159 upper=3.14159 effort=0.0 velocity=0.0
- added joint 2Link5_2Link6: type revolute, parent 2Link5, child 2Link6, origin xyz=0 0 0.5 rpy=0 0 0, axis 1 1 0, limit lower=-3.14159 upper=3.14159 effort=0.0 velocity=0.0
- added joint 2Link6_2Link7: type revolute, parent 2Link6, child 2Link7, origin xyz=0 0 0.5 rpy=0 0 0, axis 1 1 0, limit lower=-3.14159 upper=3.14159 effort=0.0 velocity=0.0
- added joint 3Link0_3Link1: type revolute, parent 3Link0, child 3Link1, origin xyz=0.5 0 0 rpy=0 0 0, axis 1 1 0, limit lower=-3.14159 upper=3.14159 effort=0.0 velocity=0.0
- added joint 3Link1_3Link2: type revolute, parent 3Link1, child 3Link2, origin xyz=0.5 0 0 rpy=0 0 0, axis 1 1 0, limit lower=-3.14159 upper=3.14159 effort=0.0 velocity=0.0
- added joint 3Link2_3Link3: type revolute, parent 3Link2, child 3Link3, origin xyz=0.5 0 0 rpy=0 0 0, axis 1 1 0, limit lower=-3.14159 upper=3.14159 effort=0.0 velocity=0.0
- added joint 3Link3_3Link4: type revolute, parent 3Link3, child 3Link4, origin xyz=0.5 0 0 rpy=0 0 0, axis 1 1 0, limit lower=-3.14159 upper=3.14159 effort=0.0 velocity=0.0
- added joint 3Link4_3Link5: type revolute, parent 3Link4, child 3Link5, origin xyz=0.5 0 0 rpy=0 0 0, axis 1 1 0, limit lower=-3.14159 upper=3.14159 effort=0.0 velocity=0.0
- added joint 3Link5_3Link6: type revolute, parent 3Link5, child 3Link6, origin xyz=0.5 0 0 rpy=0 0 0, axis 1 1 0, limit lower=-3.14159 upper=3.14159 effort=0.0 velocity=0.0
- added joint 3Link6_3Link7: type revolute, parent 3Link6, child 3Link7, origin xyz=0.5 0 0 rpy=0 0 0, axis 1 1 0, limit lower=-3.14159 upper=3.14159 effort=0.0 velocity=0.0
- added joint 3Link7_3Link8: type revolute, parent 3Link7, child 3Link8, origin xyz=0.5 0 0 rpy=0 0 0, axis 1 1 0, limit lower=-3.14159 upper=3.14159 effort=0.0 velocity=0.0
- added joint 4Link0_4Link1: type revolute, parent 4Link0, child 4Link1, origin xyz=0 -0.5 0 rpy=0 0 0, axis 1 1 0, limit lower=-3.14159 upper=3.14159 effort=0.0 velocity=0.0
- added joint 4Link1_4Link2: type revolute, parent 4Link1, child 4Link2, origin xyz=0 -0.5 0 rpy=0 0 0, axis 1 1 0, limit lower=-3.14159 upper=3.14159 effort=0.0 velocity=0.0
- added joint 4Link2_4Link3: type revolute, parent 4Link2, child 4Link3, origin xyz=0 -0.5 0 rpy=0 0 0, axis 1 1 0, limit lower=-3.14159 upper=3.14159 effort=0.0 velocity=0.0
- added joint 4Link3_4Link4: type revolute, parent 4Link3, child 4Link4, origin xyz=0 -0.5 0 rpy=0 0 0, axis 1 1 0, limit lower=-3.14159 upper=3.14159 effort=0.0 velocity=0.0
- added joint 4Link4_4Link5: type revolute, parent 4Link4, child 4Link5, origin xyz=0 -0.5 0 rpy=0 0 0, axis 1 1 0, limit lower=-3.14159 upper=3.14159 effort=0.0 velocity=0.0
- added joint 4Link5_4Link6: type revolute, parent 4Link5, child 4Link6, origin xyz=0 -0.5 0 rpy=0 0 0, axis 1 1 0, limit lower=-3.14159 upper=3.14159 effort=0.0 velocity=0.0
- added joint 4Link6_4Link7: type revolute, parent 4Link6, child 4Link7, origin xyz=0 -0.5 0 rpy=0 0 0, axis 1 1 0, limit lower=-3.14159 upper=3.14159 effort=0.0 velocity=0.0
- added joint 4Link7_4Link8: type revolute, parent 4Link7, child 4Link8, origin xyz=0 -0.5 0 rpy=0 0 0, axis 1 1 0, limit lower=-3.14159 upper=3.14159 effort=0.0 velocity=0.0
- added joint 4Link8_4Link9: type revolute, parent 4Link8, child 4Link9, origin xyz=0 -0.5 0 rpy=0 0 0, axis 1 1 0, limit lower=-3.14159 upper=3.14159 effort=0.0 velocity=0.0
- added joint Torso_0Link0: type revolute, parent Torso, child 0Link0, origin xyz=0.0 2.0 9.5 rpy=0 0 0, axis 1 1 0, limit lower=-3.14159 upper=3.14159 effort=0.0 velocity=0.0
- added joint Torso_1Link0: type revolute, parent Torso, child 1Link0, origin xyz=-0.5 2.0 10.0 rpy=0 0 0, axis 1 1 0, limit lower=-3.14159 upper=3.14159 effort=0.0 velocity=0.0
- added joint Torso_2Link0: type revolute, parent Torso, child 2Link0, origin xyz=0.0 2.0 10.5 rpy=0 0 0, axis 1 1 0, limit lower=-3.14159 upper=3.14159 effort=0.0 velocity=0.0
- added joint Torso_3Link0: type revolute, parent Torso, child 3Link0, origin xyz=0.5 2.0 10.0 rpy=0 0 0, axis 1 1 0, limit lower=-3.14159 upper=3.14159 effort=0.0 velocity=0.0
- added joint Torso_4Link0: type revolute, parent Torso, child 4Link0, origin xyz=0.0 1.5 10.0 rpy=0 0 0, axis 1 1 0, limit lower=-3.14159 upper=3.14159 effort=0.0 velocity=0.0
