Commit message: readme

File: body.urdf (robot description, URDF)
Before this commit: robot robot, 48 links, 47 joints
Links:
- removed link 3Link8
- removed link 4Link8
- removed link 4Link9
- added link 1Link10, mass 1; collision box size=0.5028903666952979 0.5197577056685698 0.6364339202927125; visual box size=0.5028903666952979 0.5197577056685698 0.6364339202927125
- added link 1Link11, mass 1; collision box size=0.1655832738071138 0.062220421405704496 0.9402335033325296; visual box size=0.1655832738071138 0.062220421405704496 0.9402335033325296
- added link 1Link9, mass 1; collision box size=0.33657480715807075 0.6076420165772435 0.3236386235675969; visual box size=0.33657480715807075 0.6076420165772435 0.3236386235675969
- added link 2Link10, mass 1; collision box size=0.5237561634064698 0.7319461608083467 0.03804997626069939; visual box size=0.5237561634064698 0.7319461608083467 0.03804997626069939
- added link 2Link8, mass 1; collision box size=0.16785348622126328 0.0682709224526814 0.9826973359727801; visual box size=0.16785348622126328 0.0682709224526814 0.9826973359727801
- added link 2Link9, mass 1; collision box size=0.448332259115354 0.6255022898198999 0.4432979107264786; visual box size=0.448332259115354 0.6255022898198999 0.4432979107264786
- added link 5Link0, mass 1; collision box size=0.6457776413718429 0.2794439310567095 0.9268688423156197; visual box size=0.6457776413718429 0.2794439310567095 0.9268688423156197
- added link 5Link1, mass 1; collision box size=0.49183337535218896 0.8692332642677268 0.5495771579097899; visual box size=0.49183337535218896 0.8692332642677268 0.5495771579097899
- added link 5Link10, mass 1; collision box size=0.17790324577182426 0.5773180226418729 0.8134786761245398; visual box size=0.17790324577182426 0.5773180226418729 0.8134786761245398
- added link 5Link2, mass 1; collision box size=0.018640126755856357 0.7929524023843806 0.6057203801936355; visual box size=0.018640126755856357 0.7929524023843806 0.6057203801936355
- added link 5Link3, mass 1; collision box size=0.49145921408666926 0.9153241321822438 0.14976195019046645; visual box size=0.49145921408666926 0.9153241321822438 0.14976195019046645
- added link 5Link4, mass 1; collision box size=0.8858913781413886 0.2160083476563036 0.8069575072808313; visual box size=0.8858913781413886 0.2160083476563036 0.8069575072808313
- added link 5Link5, mass 1; collision box size=0.7839003179466572 0.5963494863835547 0.5070259099517069; visual box size=0.7839003179466572 0.5963494863835547 0.5070259099517069
- added link 5Link6, mass 1; collision box size=0.37635137525006335 0.4922922621800063 0.5077524124795836; visual box size=0.37635137525006335 0.4922922621800063 0.5077524124795836
- added link 5Link7, mass 1; collision box size=0.2880666801391121 0.09441240557504771 0.5087000416435181; visual box size=0.2880666801391121 0.09441240557504771 0.5087000416435181
- added link 5Link8, mass 1; collision box size=0.2178229266282773 0.04711588224994412 0.02059716703456449; visual box size=0.2178229266282773 0.04711588224994412 0.02059716703456449
- added link 5Link9, mass 1; collision box size=0.509845583527544 0.22437658035560737 0.5820272615799689; visual box size=0.509845583527544 0.22437658035560737 0.5820272615799689
- link 0Link0: geometry collision box size=0.35853525612280046 0.023169419879083053 0.9081941626735217; visual box size=0.35853525612280046 0.023169419879083053 0.9081941626735217
- link 0Link1: geometry collision box size=0.6369423790539585 0.49652467301791336 0.01768629470343852; visual box size=0.6369423790539585 0.49652467301791336 0.01768629470343852
- link 0Link10: geometry collision box size=0.26863896701240686 0.49420769881648086 0.9315517120916973; visual box size=0.26863896701240686 0.49420769881648086 0.9315517120916973
- link 0Link2: geometry collision box size=0.13939395564319812 0.7527476207740394 0.26577621897160353; visual box size=0.13939395564319812 0.7527476207740394 0.26577621897160353
- link 0Link3: geometry collision box size=0.6496650511676053 0.26522459492077843 0.3714044234098257; visual box size=0.6496650511676053 0.26522459492077843 0.3714044234098257
- link 0Link4: geometry collision box size=0.1523805466114162 0.21625772763736184 0.4686265617731097; visual box size=0.1523805466114162 0.21625772763736184 0.4686265617731097
- link 0Link5: geometry collision box size=0.49946874373714556 0.908081373669752 0.7911336315930636; visual box size=0.49946874373714556 0.908081373669752 0.7911336315930636
- link 0Link6: geometry collision box size=0.643251595032799 0.542514943673118 0.534149563561826; visual box size=0.643251595032799 0.542514943673118 0.534149563561826
- link 0Link7: geometry collision box size=0.06917704508814404 0.587047153302547 0.2531115561053242; visual box size=0.06917704508814404 0.587047153302547 0.2531115561053242
- link 0Link8: geometry collision box size=0.7125340761093377 0.6345828839086319 0.06433469293588256; visual box size=0.7125340761093377 0.6345828839086319 0.06433469293588256
- link 0Link9: geometry collision box size=0.5553448214027334 0.5213487075256407 0.01952659126090328; visual box size=0.5553448214027334 0.5213487075256407 0.01952659126090328
- link 1Link0: geometry collision box size=0.12814093847072017 0.438849244641043 0.1156440647024578; visual box size=0.12814093847072017 0.438849244641043 0.1156440647024578
- link 1Link1: geometry collision box size=0.19677177560712078 0.2930126617584009 0.8435923691385357; visual box size=0.19677177560712078 0.2930126617584009 0.8435923691385357
- link 1Link2: geometry collision box size=0.5710029773298687 0.17076076435950616 0.6809994310548366; visual box size=0.5710029773298687 0.17076076435950616 0.6809994310548366
- link 1Link3: geometry collision box size=0.1197108920687201 0.41744212204321884 0.9233724606239311; visual box size=0.1197108920687201 0.41744212204321884 0.9233724606239311
- link 1Link4: geometry collision box size=0.4971284200960371 0.7657829491370695 0.051994923802653914; visual box size=0.4971284200960371 0.7657829491370695 0.051994923802653914
- link 1Link5: geometry collision box size=0.38567881917171243 0.4918423688385043 0.5495278755631345; visual box size=0.38567881917171243 0.4918423688385043 0.5495278755631345
- link 1Link6: geometry collision box size=0.24801839291230743 0.7985877718297347 0.4611784884416984; visual box size=0.24801839291230743 0.7985877718297347 0.4611784884416984
- link 1Link7: geometry collision box size=0.6772432956952605 0.5226892193562412 0.5624973526479816; visual box size=0.6772432956952605 0.5226892193562412 0.5624973526479816
- link 1Link8: geometry collision box size=0.7681398483237429 0.517234023985469 0.6833089341288957; visual box size=0.7681398483237429 0.517234023985469 0.6833089341288957
- link 2Link0: geometry collision box size=0.641706610589876 0.41911820665750676 0.5680637309629364; visual box size=0.641706610589876 0.41911820665750676 0.5680637309629364
- link 2Link1: geometry collision box size=0.22746831773489584 0.44867101268780807 0.13212552098685038; visual box size=0.22746831773489584 0.44867101268780807 0.13212552098685038
- link 2Link2: geometry collision box size=0.8853836234908758 0.5104728092280595 0.5845808247831674; visual box size=0.8853836234908758 0.5104728092280595 0.5845808247831674
- link 2Link3: geometry collision box size=0.7537968989923759 0.16174046042151324 0.8308122982428593; visual box size=0.7537968989923759 0.16174046042151324 0.8308122982428593
- link 2Link4: geometry collision box size=0.0031902243010787368 0.2720848244772769 0.35582186242423897; visual box size=0.0031902243010787368 0.2720848244772769 0.35582186242423897
- link 2Link5: geometry collision box size=0.14905950105048948 0.9887317451667764 0.32820094289999713; visual box size=0.14905950105048948 0.9887317451667764 0.32820094289999713
- link 2Link6: geometry collision box size=0.5360128064352674 0.42254189076915194 0.02955780369718164; visual box size=0.5360128064352674 0.42254189076915194 0.02955780369718164
- link 2Link7: geometry collision box size=0.2187452361649641 0.4535315719722489 0.8462552635401116; visual box size=0.2187452361649641 0.4535315719722489 0.8462552635401116
- link 3Link0: geometry collision box size=0.3162626547591556 0.911380808148886 0.3723232976176116; visual box size=0.3162626547591556 0.911380808148886 0.3723232976176116
- link 3Link1: geometry collision box size=0.06406265324895144 0.6727076254949854 0.6850880734067796; visual box size=0.06406265324895144 0.6727076254949854 0.6850880734067796
- link 3Link2: geometry collision box size=0.6352413431562342 0.6624794514843193 0.16903511025557494; visual box size=0.6352413431562342 0.6624794514843193 0.16903511025557494
- link 3Link3: geometry collision box size=0.6397875880315769 0.8886713985202491 0.8930351593564106; visual box size=0.6397875880315769 0.8886713985202491 0.8930351593564106
- link 3Link4: geometry collision box size=0.6790889576981444 0.1275538004551885 0.9144431225724055; visual box size=0.6790889576981444 0.1275538004551885 0.9144431225724055
- link 3Link5: geometry collision box size=0.17511347291830182 0.9567362244829888 0.8760993092967383; visual box size=0.17511347291830182 0.9567362244829888 0.8760993092967383
- link 3Link6: geometry collision box size=0.10110404126750605 0.34451695847896824 0.8745688050957389; visual box size=0.10110404126750605 0.34451695847896824 0.8745688050957389
- link 3Link7: geometry collision box size=0.6225956371626786 0.734536714235664 0.5764382402103841; visual box size=0.6225956371626786 0.734536714235664 0.5764382402103841
- link 4Link0: geometry collision box size=0.6579123672078686 0.8239955678907515 0.741373976510604; visual box size=0.6579123672078686 0.8239955678907515 0.741373976510604
- link 4Link1: geometry collision box size=0.2770297372768332 0.800355944866321 0.5523414242360247; visual box size=0.2770297372768332 0.800355944866321 0.5523414242360247
- link 4Link2: geometry collision box size=0.5086388323222989 0.8747462944342305 0.29857273596645295; visual box size=0.5086388323222989 0.8747462944342305 0.29857273596645295
- link 4Link3: geometry collision box size=0.26571953561180706 0.2840781788271117 0.3611837263551865; visual box size=0.26571953561180706 0.2840781788271117 0.3611837263551865
- link 4Link4: geometry collision box size=0.48100683524056453 0.3336514468737878 0.21029036457208194; visual box size=0.48100683524056453 0.3336514468737878 0.21029036457208194
- link 4Link5: geometry collision box size=0.400001885924658 0.3246924649510575 0.15177785006920996; visual box size=0.400001885924658 0.3246924649510575 0.15177785006920996
- link 4Link6: geometry collision box size=0.5736959127693169 0.6992668953224034 0.3556390805213334; visual box size=0.5736959127693169 0.6992668953224034 0.3556390805213334
- link 4Link7: geometry collision box size=0.4000198292917492 0.564122017259448 0.6647790658289567; visual box size=0.4000198292917492 0.564122017259448 0.6647790658289567
Joints:
- removed joint 3Link7_3Link8
- removed joint 4Link7_4Link8
- removed joint 4Link8_4Link9
- added joint 1Link10_1Link11: type revolute, parent 1Link10, child 1Link11, origin xyz=-0.5 0 0 rpy=0 0 0, axis 1 1 0, limit lower=-3.14159 upper=3.14159 effort=0.0 velocity=0.0
- added joint 1Link8_1Link9: type revolute, parent 1Link8, child 1Link9, origin xyz=-0.5 0 0 rpy=0 0 0, axis 1 1 0, limit lower=-3.14159 upper=3.14159 effort=0.0 velocity=0.0
- added joint 1Link9_1Link10: type revolute, parent 1Link9, child 1Link10, origin xyz=-0.5 0 0 rpy=0 0 0, axis 1 1 0, limit lower=-3.14159 upper=3.14159 effort=0.0 velocity=0.0
- added joint 2Link7_2Link8: type revolute, parent 2Link7, child 2Link8, origin xyz=0 0 0.5 rpy=0 0 0, axis 1 1 0, limit lower=-3.14159 upper=3.14159 effort=0.0 velocity=0.0
- added joint 2Link8_2Link9: type revolute, parent 2Link8, child 2Link9, origin xyz=0 0 0.5 rpy=0 0 0, axis 1 1 0, limit lower=-3.14159 upper=3.14159 effort=0.0 velocity=0.0
- added joint 2Link9_2Link10: type revolute, parent 2Link9, child 2Link10, origin xyz=0 0 0.5 rpy=0 0 0, axis 1 1 0, limit lower=-3.14159 upper=3.14159 effort=0.0 velocity=0.0
- added joint 5Link0_5Link1: type revolute, parent 5Link0, child 5Link1, origin xyz=0 0.5 0 rpy=0 0 0, axis 1 1 0, limit lower=-3.14159 upper=3.14159 effort=0.0 velocity=0.0
- added joint 5Link1_5Link2: type revolute, parent 5Link1, child 5Link2, origin xyz=0 0.5 0 rpy=0 0 0, axis 1 1 0, limit lower=-3.14159 upper=3.14159 effort=0.0 velocity=0.0
- added joint 5Link2_5Link3: type revolute, parent 5Link2, child 5Link3, origin xyz=0 0.5 0 rpy=0 0 0, axis 1 1 0, limit lower=-3.14159 upper=3.14159 effort=0.0 velocity=0.0
- added joint 5Link3_5Link4: type revolute, parent 5Link3, child 5Link4, origin xyz=0 0.5 0 rpy=0 0 0, axis 1 1 0, limit lower=-3.14159 upper=3.14159 effort=0.0 velocity=0.0
- added joint 5Link4_5Link5: type revolute, parent 5Link4, child 5Link5, origin xyz=0 0.5 0 rpy=0 0 0, axis 1 1 0, limit lower=-3.14159 upper=3.14159 effort=0.0 velocity=0.0
- added joint 5Link5_5Link6: type revolute, parent 5Link5, child 5Link6, origin xyz=0 0.5 0 rpy=0 0 0, axis 1 1 0, limit lower=-3.14159 upper=3.14159 effort=0.0 velocity=0.0
- added joint 5Link6_5Link7: type revolute, parent 5Link6, child 5Link7, origin xyz=0 0.5 0 rpy=0 0 0, axis 1 1 0, limit lower=-3.14159 upper=3.14159 effort=0.0 velocity=0.0
- added joint 5Link7_5Link8: type revolute, parent 5Link7, child 5Link8, origin xyz=0 0.5 0 rpy=0 0 0, axis 1 1 0, limit lower=-3.14159 upper=3.14159 effort=0.0 velocity=0.0
- added joint 5Link8_5Link9: type revolute, parent 5Link8, child 5Link9, origin xyz=0 0.5 0 rpy=0 0 0, axis 1 1 0, limit lower=-3.14159 upper=3.14159 effort=0.0 velocity=0.0
- added joint 5Link9_5Link10: type revolute, parent 5Link9, child 5Link10, origin xyz=0 0.5 0 rpy=0 0 0, axis 1 1 0, limit lower=-3.14159 upper=3.14159 effort=0.0 velocity=0.0
- added joint Torso_5Link0: type revolute, parent Torso, child 5Link0, origin xyz=0.0 2.5 10.0 rpy=0 0 0, axis 1 1 0, limit lower=-3.14159 upper=3.14159 effort=0.0 velocity=0.0
