Commit message: final v1

File: body.urdf (robot description, URDF)
Before this commit: robot robot, 62 links, 61 joints
Links:
- removed link 1Link11
- removed link 2Link10
- removed link 2Link8
- removed link 2Link9
- removed link 5Link0
- removed link 5Link1
- removed link 5Link10
- removed link 5Link2
- removed link 5Link3
- removed link 5Link4
- removed link 5Link5
- removed link 5Link6
- removed link 5Link7
- removed link 5Link8
- removed link 5Link9
- added link 0Link11, mass 1; collision box size=0.7662265931177182 0.8305010888744477 0.043201508947181444; visual box size=0.7662265931177182 0.8305010888744477 0.043201508947181444
- added link 3Link10, mass 1; collision box size=0.46410630533515107 0.12093015119984751 0.26879031245766516; visual box size=0.46410630533515107 0.12093015119984751 0.26879031245766516
- added link 3Link8, mass 1; collision box size=0.2745131727659015 0.8224906715234093 0.5442424775752976; visual box size=0.2745131727659015 0.8224906715234093 0.5442424775752976
- added link 3Link9, mass 1; collision box size=0.6219825017625058 0.302943343817206 0.07426497804999665; visual box size=0.6219825017625058 0.302943343817206 0.07426497804999665
- added link 4Link8, mass 1; collision box size=0.9669098499258859 0.5897205612650378 0.1847049851342767; visual box size=0.9669098499258859 0.5897205612650378 0.1847049851342767
- added link 4Link9, mass 1; collision box size=0.9232053636061093 0.6448526507076447 0.04766493224167201; visual box size=0.9232053636061093 0.6448526507076447 0.04766493224167201
- link 0Link0: geometry collision box size=0.8391906626935169 0.5312167122613297 0.9980467590666072; visual box size=0.8391906626935169 0.5312167122613297 0.9980467590666072
- link 0Link1: geometry collision box size=0.23852779133092927 0.3757720104922069 0.39188842817764946; visual box size=0.23852779133092927 0.3757720104922069 0.39188842817764946
- link 0Link10: geometry collision box size=0.8391394381083811 0.03983965033478931 0.747043842013903; visual box size=0.8391394381083811 0.03983965033478931 0.747043842013903
- link 0Link2: geometry collision box size=0.3521608622913115 0.6891258671667737 0.0928104059763708; visual box size=0.3521608622913115 0.6891258671667737 0.0928104059763708
- link 0Link3: geometry collision box size=0.4028210693243973 0.21684853571936458 0.02097241571987174; visual box size=0.4028210693243973 0.21684853571936458 0.02097241571987174
- link 0Link4: geometry collision box size=0.24393573175186456 0.30241578227133636 0.31066472075063967; visual box size=0.24393573175186456 0.30241578227133636 0.31066472075063967
- link 0Link5: geometry collision box size=0.1249147455907802 0.23972026720370299 0.8101907449731642; visual box size=0.1249147455907802 0.23972026720370299 0.8101907449731642
- link 0Link6: geometry collision box size=0.22106313892194196 0.48863500152944594 0.9871246310572794; visual box size=0.22106313892194196 0.48863500152944594 0.9871246310572794
- link 0Link7: geometry collision box size=0.5453183136311245 0.8053505869594568 0.6403208637061103; visual box size=0.5453183136311245 0.8053505869594568 0.6403208637061103
- link 0Link8: geometry collision box size=0.19711120484219224 0.8453253803443892 0.4090933661035141; visual box size=0.19711120484219224 0.8453253803443892 0.4090933661035141
- link 0Link9: geometry collision box size=0.9439241805122842 0.7480928087636789 0.17921972527730257; visual box size=0.9439241805122842 0.7480928087636789 0.17921972527730257
- link 1Link0: geometry collision box size=0.512863349789045 0.20312941826098008 0.3187347982219608; visual box size=0.512863349789045 0.20312941826098008 0.3187347982219608
- link 1Link1: geometry collision box size=0.614469749094057 0.4546817788820552 0.8654131205798931; visual box size=0.614469749094057 0.4546817788820552 0.8654131205798931
- link 1Link10: geometry collision box size=0.275555569770636 0.0522928130597472 0.8937907632234283; visual box size=0.275555569770636 0.0522928130597472 0.8937907632234283
- link 1Link2: geometry collision box size=0.8263681072359923 0.7047961110932512 0.5601788386020392; visual box size=0.8263681072359923 0.7047961110932512 0.5601788386020392
- link 1Link3: geometry collision box size=0.652281436872417 0.7742332389449488 0.7714124738666526; visual box size=0.652281436872417 0.7742332389449488 0.7714124738666526
- link 1Link4: geometry collision box size=0.25707921963899427 0.8767391431360416 0.8583433472416583; visual box size=0.25707921963899427 0.8767391431360416 0.8583433472416583
- link 1Link5: geometry collision box size=0.23560159428954586 0.2700487966096091 0.9830580422685679; visual box size=0.23560159428954586 0.2700487966096091 0.9830580422685679
- link 1Link6: geometry collision box size=0.23723001433127444 0.38455160715857073 0.6601490189191811; visual box size=0.23723001433127444 0.38455160715857073 0.6601490189191811
- link 1Link7: geometry collision box size=0.0744076315575547 0.9640324858180067 0.8006088083639696; visual box size=0.0744076315575547 0.9640324858180067 0.8006088083639696
- link 1Link8: geometry collision box size=0.09220540822836232 0.02245197912407726 0.38773007229704315; visual box size=0.09220540822836232 0.02245197912407726 0.38773007229704315
- link 1Link9: geometry collision box size=0.8656033756045215 0.4578479931588475 0.2907510082255098; visual box size=0.8656033756045215 0.4578479931588475 0.2907510082255098
- link 2Link0: geometry collision box size=0.23784127610810957 0.6661400086149362 0.20386364947666435; visual box size=0.23784127610810957 0.6661400086149362 0.20386364947666435
- link 2Link1: geometry collision box size=0.7292464856714037 0.6011673511943688 0.908072806867357; visual box size=0.7292464856714037 0.6011673511943688 0.908072806867357
- link 2Link2: geometry collision box size=0.23424886107318932 0.460140878242561 0.1212202954733731; visual box size=0.23424886107318932 0.460140878242561 0.1212202954733731
- link 2Link3: geometry collision box size=0.2536674328031673 0.9252924689335668 0.05800482566694165; visual box size=0.2536674328031673 0.9252924689335668 0.05800482566694165
- link 2Link4: geometry collision box size=0.44103076707269007 0.2905708799536548 0.004839363302910127; visual box size=0.44103076707269007 0.2905708799536548 0.004839363302910127
- link 2Link5: geometry collision box size=0.29054798940659243 0.36640691958862204 0.5443149242125256; visual box size=0.29054798940659243 0.36640691958862204 0.5443149242125256
- link 2Link6: geometry collision box size=0.776164258589635 0.705968378149732 0.9950619259979407; visual box size=0.776164258589635 0.705968378149732 0.9950619259979407
- link 2Link7: geometry collision box size=0.31679042321547557 0.6175764029066443 0.1946553901949981; visual box size=0.31679042321547557 0.6175764029066443 0.1946553901949981
- link 3Link0: geometry collision box size=0.7854672518587498 0.26697651261965316 0.48305170847730217; visual box size=0.7854672518587498 0.26697651261965316 0.48305170847730217
- link 3Link1: geometry collision box size=0.7496240663326561 0.08123180528259022 0.5116647354347204; visual box size=0.7496240663326561 0.08123180528259022 0.5116647354347204
- link 3Link2: geometry collision box size=0.4687158662771459 0.04045529506361978 0.31116067515825985; visual box size=0.4687158662771459 0.04045529506361978 0.31116067515825985
- link 3Link3: geometry collision box size=0.9008906073110642 0.3269679967388536 0.7829790128344977; visual box size=0.9008906073110642 0.3269679967388536 0.7829790128344977
- link 3Link4: geometry collision box size=0.053179988204543616 0.09459118893263851 0.4749545957997202; visual box size=0.053179988204543616 0.09459118893263851 0.4749545957997202
- link 3Link5: geometry collision box size=0.24715876499988332 0.16591483685311503 0.875779228989194; visual box size=0.24715876499988332 0.16591483685311503 0.875779228989194
- link 3Link6: geometry collision box size=0.5493021972432666 0.8354650201152135 0.8702630158347419; visual box size=0.5493021972432666 0.8354650201152135 0.8702630158347419
- link 3Link7: geometry collision box size=0.2418984708635169 0.13177037914682743 0.35552712705543543; visual box size=0.2418984708635169 0.13177037914682743 0.35552712705543543
- link 4Link0: geometry collision box size=0.9220094932828626 0.679084546468696 0.5576934528407631; visual box size=0.9220094932828626 0.679084546468696 0.5576934528407631
- link 4Link1: geometry collision box size=0.2908091492584536 0.11702296599300355 0.5832460879981264; visual box size=0.2908091492584536 0.11702296599300355 0.5832460879981264
- link 4Link2: geometry collision box size=0.7037316083883449 0.3726130669287171 0.45962544104259095; visual box size=0.7037316083883449 0.3726130669287171 0.45962544104259095
- link 4Link3: geometry collision box size=0.07487388935689399 0.936624108151276 0.9758238250811906; visual box size=0.07487388935689399 0.936624108151276 0.9758238250811906
- link 4Link4: geometry collision box size=0.29143805561881764 0.8757175433939255 0.389287084907907; visual box size=0.29143805561881764 0.8757175433939255 0.389287084907907
- link 4Link5: geometry collision box size=0.7060892397298315 0.5410192990543596 0.43214405558221936; visual box size=0.7060892397298315 0.5410192990543596 0.43214405558221936
- link 4Link6: geometry collision box size=0.1418699914893814 0.4856243561416391 0.3829512338119727; visual box size=0.1418699914893814 0.4856243561416391 0.3829512338119727
- link 4Link7: geometry collision box size=0.5146999156756028 0.4919640999485192 0.13263230167691986; visual box size=0.5146999156756028 0.4919640999485192 0.13263230167691986
Joints:
- removed joint 1Link10_1Link11
- removed joint 2Link7_2Link8
- removed joint 2Link8_2Link9
- removed joint 2Link9_2Link10
- removed joint 5Link0_5Link1
- removed joint 5Link1_5Link2
- removed joint 5Link2_5Link3
- removed joint 5Link3_5Link4
- removed joint 5Link4_5Link5
- removed joint 5Link5_5Link6
- removed joint 5Link6_5Link7
- removed joint 5Link7_5Link8
- removed joint 5Link8_5Link9
- removed joint 5Link9_5Link10
- removed joint Torso_5Link0
- added joint 0Link10_0Link11: type revolute, parent 0Link10, child 0Link11, origin xyz=0 0 -0.5 rpy=0 0 0, axis 1 1 0, limit lower=-3.14159 upper=3.14159 effort=0.0 velocity=0.0
- added joint 3Link7_3Link8: type revolute, parent 3Link7, child 3Link8, origin xyz=0.5 0 0 rpy=0 0 0, axis 1 1 0, limit lower=-3.14159 upper=3.14159 effort=0.0 velocity=0.0
- added joint 3Link8_3Link9: type revolute, parent 3Link8, child 3Link9, origin xyz=0.5 0 0 rpy=0 0 0, axis 1 1 0, limit lower=-3.14159 upper=3.14159 effort=0.0 velocity=0.0
- added joint 3Link9_3Link10: type revolute, parent 3Link9, child 3Link10, origin xyz=0.5 0 0 rpy=0 0 0, axis 1 1 0, limit lower=-3.14159 upper=3.14159 effort=0.0 velocity=0.0
- added joint 4Link7_4Link8: type revolute, parent 4Link7, child 4Link8, origin xyz=0 -0.5 0 rpy=0 0 0, axis 1 1 0, limit lower=-3.14159 upper=3.14159 effort=0.0 velocity=0.0
- added joint 4Link8_4Link9: type revolute, parent 4Link8, child 4Link9, origin xyz=0 -0.5 0 rpy=0 0 0, axis 1 1 0, limit lower=-3.14159 upper=3.14159 effort=0.0 velocity=0.0
