Commit message: etc

File: body.urdf (robot description, URDF)
Before this commit: robot robot, 53 links, 52 joints
Links:
- removed link 0Link11
- removed link 3Link10
- added link 1Link11, mass 1; collision box size=0.17337400800014102 0.8101104125838506 0.19556140580324488; visual box size=0.17337400800014102 0.8101104125838506 0.19556140580324488
- added link 2Link8, mass 1; collision box size=0.2349117255643306 0.5155540311475925 0.914116711134303; visual box size=0.2349117255643306 0.5155540311475925 0.914116711134303
- added link 5Link0, mass 1; collision box size=0.9295780510834669 0.6135614578754535 0.2885802776747428; visual box size=0.9295780510834669 0.6135614578754535 0.2885802776747428
- added link 5Link1, mass 1; collision box size=0.9782128570144072 0.6815083192956277 0.9714792795977119; visual box size=0.9782128570144072 0.6815083192956277 0.9714792795977119
- added link 5Link10, mass 1; collision box size=0.09030567879021678 0.5078908985215251 0.11515067385441602; visual box size=0.09030567879021678 0.5078908985215251 0.11515067385441602
- added link 5Link2, mass 1; collision box size=0.9787919056094412 0.6331631871651937 0.06755529613086464; visual box size=0.9787919056094412 0.6331631871651937 0.06755529613086464
- added link 5Link3, mass 1; collision box size=0.8822830351808891 0.3268443541741579 0.2686530382805854; visual box size=0.8822830351808891 0.3268443541741579 0.2686530382805854
- added link 5Link4, mass 1; collision box size=0.7302646640918424 0.5041898793190218 0.5845335363465434; visual box size=0.7302646640918424 0.5041898793190218 0.5845335363465434
- added link 5Link5, mass 1; collision box size=0.5949530278532691 0.47336386487493853 0.5715525585729602; visual box size=0.5949530278532691 0.47336386487493853 0.5715525585729602
- added link 5Link6, mass 1; collision box size=0.7278775103831042 0.831499456246229 0.3661163015786517; visual box size=0.7278775103831042 0.831499456246229 0.3661163015786517
- added link 5Link7, mass 1; collision box size=0.07593135370792292 0.289443261165795 0.6875557625222005; visual box size=0.07593135370792292 0.289443261165795 0.6875557625222005
- added link 5Link8, mass 1; collision box size=0.3739625907294082 0.014475604547341647 0.4597053944315689; visual box size=0.3739625907294082 0.014475604547341647 0.4597053944315689
- added link 5Link9, mass 1; collision box size=0.8706646368512404 0.22847213626759721 0.19608604375412808; visual box size=0.8706646368512404 0.22847213626759721 0.19608604375412808
- link 0Link0: geometry collision box size=0.7657147413993838 0.4018900349727247 0.19118644739719148; visual box size=0.7657147413993838 0.4018900349727247 0.19118644739719148
- link 0Link1: geometry collision box size=0.6683952000082469 0.3755767381684425 0.5947791175966025; visual box size=0.6683952000082469 0.3755767381684425 0.5947791175966025
- link 0Link10: geometry collision box size=0.4125674847270916 0.7850601995080021 0.5302688108499193; visual box size=0.4125674847270916 0.7850601995080021 0.5302688108499193
- link 0Link2: geometry collision box size=0.601296626784739 0.3540649492150869 0.39249812953995356; visual box size=0.601296626784739 0.3540649492150869 0.39249812953995356
- link 0Link3: geometry collision box size=0.49445200025860225 0.9428365250291603 0.18175706683559267; visual box size=0.49445200025860225 0.9428365250291603 0.18175706683559267
- link 0Link4: geometry collision box size=0.3126474694776388 0.7146841250892996 0.10431549126595363; visual box size=0.3126474694776388 0.7146841250892996 0.10431549126595363
- link 0Link5: geometry collision box size=0.22210681864122128 0.1209243205441003 0.1223338920768623; visual box size=0.22210681864122128 0.1209243205441003 0.1223338920768623
- link 0Link6: geometry collision box size=0.019733120449502928 0.5115542458872212 0.7275630611562823; visual box size=0.019733120449502928 0.5115542458872212 0.7275630611562823
- link 0Link7: geometry collision box size=0.6527809677956634 0.12614508581119466 0.8237311864726382; visual box size=0.6527809677956634 0.12614508581119466 0.8237311864726382
- link 0Link8: geometry collision box size=0.20900144266040666 0.6356845801062496 0.5022501412308875; visual box size=0.20900144266040666 0.6356845801062496 0.5022501412308875
- link 0Link9: geometry collision box size=0.43964154570302383 0.09805171688126846 0.2925192269061493; visual box size=0.43964154570302383 0.09805171688126846 0.2925192269061493
- link 1Link0: geometry collision box size=0.35203601788342154 0.8266952334873006 0.6578477716540477; visual box size=0.35203601788342154 0.8266952334873006 0.6578477716540477
- link 1Link1: geometry collision box size=0.03941249344081499 0.19764328699619282 0.11882249311832094; visual box size=0.03941249344081499 0.19764328699619282 0.11882249311832094
- link 1Link10: geometry collision box size=0.4178612787636473 0.21510087835930536 0.5224014746838535; visual box size=0.4178612787636473 0.21510087835930536 0.5224014746838535
- link 1Link2: geometry collision box size=0.3345509432071935 0.4056297363921205 0.2054924711263021; visual box size=0.3345509432071935 0.4056297363921205 0.2054924711263021
- link 1Link3: geometry collision box size=0.9309880274286618 0.26896225807458407 0.9934712618748207; visual box size=0.9309880274286618 0.26896225807458407 0.9934712618748207
- link 1Link4: geometry collision box size=0.18607597103867235 0.7377457668457398 0.08763706474665256; visual box size=0.18607597103867235 0.7377457668457398 0.08763706474665256
- link 1Link5: geometry collision box size=0.9494855258091474 0.5461312982639455 0.6239417222029567; visual box size=0.9494855258091474 0.5461312982639455 0.6239417222029567
- link 1Link6: geometry collision box size=0.2760968989869761 0.7741939426497936 0.7227940278452608; visual box size=0.2760968989869761 0.7741939426497936 0.7227940278452608
- link 1Link7: geometry collision box size=0.2747368018619951 0.32768484092967043 0.9878306232989059; visual box size=0.2747368018619951 0.32768484092967043 0.9878306232989059
- link 1Link8: geometry collision box size=0.559071938449223 0.35464871241178086 0.985483270919331; visual box size=0.559071938449223 0.35464871241178086 0.985483270919331
- link 1Link9: geometry collision box size=0.45074251230521034 0.02532657101353375 0.38669791103245843; visual box size=0.45074251230521034 0.02532657101353375 0.38669791103245843
- link 2Link0: geometry collision box size=0.44508666908910477 0.40964758461661854 0.3623413432768209; visual box size=0.44508666908910477 0.40964758461661854 0.3623413432768209
- link 2Link1: geometry collision box size=0.12775596763662234 0.7124478234862365 0.4715488334904234; visual box size=0.12775596763662234 0.7124478234862365 0.4715488334904234
- link 2Link2: geometry collision box size=0.8730787919493201 0.270404869123014 0.6322558977417838; visual box size=0.8730787919493201 0.270404869123014 0.6322558977417838
- link 2Link3: geometry collision box size=0.13351004365365027 0.1506483667173385 0.4968611852962669; visual box size=0.13351004365365027 0.1506483667173385 0.4968611852962669
- link 2Link4: geometry collision box size=0.8426897425209593 0.21121655511015813 0.6394540114197048; visual box size=0.8426897425209593 0.21121655511015813 0.6394540114197048
- link 2Link5: geometry collision box size=0.2631862571804815 0.5785386749330771 0.46346527163476225; visual box size=0.2631862571804815 0.5785386749330771 0.46346527163476225
- link 2Link6: geometry collision box size=0.44773470231274004 0.17846365582171542 0.7014657240785622; visual box size=0.44773470231274004 0.17846365582171542 0.7014657240785622
- link 2Link7: geometry collision box size=0.8201094471658046 0.17081767561459915 0.2848349285856022; visual box size=0.8201094471658046 0.17081767561459915 0.2848349285856022
- link 3Link0: geometry collision box size=0.48620989063720255 0.38061169275151996 0.9128969287097661; visual box size=0.48620989063720255 0.38061169275151996 0.9128969287097661
- link 3Link1: geometry collision box size=0.5475319756451277 0.7420634151710377 0.7682398442770877; visual box size=0.5475319756451277 0.7420634151710377 0.7682398442770877
- link 3Link2: geometry collision box size=0.16453486711036702 0.9604911394736295 0.12503948544211207; visual box size=0.16453486711036702 0.9604911394736295 0.12503948544211207
- link 3Link3: geometry collision box size=0.7978766890562005 0.2559525848549671 0.9374636205724656; visual box size=0.7978766890562005 0.2559525848549671 0.9374636205724656
- link 3Link4: geometry collision box size=0.16973761435670864 0.8433235947628457 0.5452356720861234; visual box size=0.16973761435670864 0.8433235947628457 0.5452356720861234
- link 3Link5: geometry collision box size=0.5247571728554133 0.6811504054160347 0.24631630872012267; visual box size=0.5247571728554133 0.6811504054160347 0.24631630872012267
- link 3Link6: geometry collision box size=0.47694938288166977 0.23122655623988786 0.06202180537741464; visual box size=0.47694938288166977 0.23122655623988786 0.06202180537741464
- link 3Link7: geometry collision box size=0.5446770747075308 0.8105820243434119 0.5836190910166511; visual box size=0.5446770747075308 0.8105820243434119 0.5836190910166511
- link 3Link8: geometry collision box size=0.1690512707509928 0.622834292017902 0.4138104225763066; visual box size=0.1690512707509928 0.622834292017902 0.4138104225763066
- link 3Link9: geometry collision box size=0.1947999465029392 0.7482067150691023 0.5781248599428521; visual box size=0.1947999465029392 0.7482067150691023 0.5781248599428521
- link 4Link0: geometry collision box size=0.5786956896804863 0.5961804041664873 0.4841173526179732; visual box size=0.5786956896804863 0.5961804041664873 0.4841173526179732
- link 4Link1: geometry collision box size=0.5971069901448544 0.5283248145552921 0.5547499801987146; visual box size=0.5971069901448544 0.5283248145552921 0.5547499801987146
- link 4Link2: geometry collision box size=0.9138947466946364 0.9657060991122325 0.9526145794221627; visual box size=0.9138947466946364 0.9657060991122325 0.9526145794221627
- link 4Link3: geometry collision box size=0.2302394192039685 0.07551261460739944 0.8187212873965031; visual box size=0.2302394192039685 0.07551261460739944 0.8187212873965031
- link 4Link4: geometry collision box size=0.7076090948709283 0.17387604312680693 0.7588877210890649; visual box size=0.7076090948709283 0.17387604312680693 0.7588877210890649
- link 4Link5: geometry collision box size=0.720589709100226 0.6093338353565789 0.4430116391332358; visual box size=0.720589709100226 0.6093338353565789 0.4430116391332358
- link 4Link6: geometry collision box size=0.5698671739992436 0.2632293329290324 0.7918084402802381; visual box size=0.5698671739992436 0.2632293329290324 0.7918084402802381
- link 4Link7: geometry collision box size=0.9785035350715917 0.22640348144203948 0.3577314006314386; visual box size=0.9785035350715917 0.22640348144203948 0.3577314006314386
- link 4Link8: geometry collision box size=0.7404127347006311 0.293643095065123 0.49129794743781574; visual box size=0.7404127347006311 0.293643095065123 0.49129794743781574
- link 4Link9: geometry collision box size=0.28521626511272946 0.7411320129225034 0.48153066853534676; visual box size=0.28521626511272946 0.7411320129225034 0.48153066853534676
Joints:
- removed joint 0Link10_0Link11
- removed joint 3Link9_3Link10
- added joint 1Link10_1Link11: type revolute, parent 1Link10, child 1Link11, origin xyz=-0.5 0 0 rpy=0 0 0, axis 1 1 0, limit lower=-3.14159 upper=3.14159 effort=0.0 velocity=0.0
- added joint 2Link7_2Link8: type revolute, parent 2Link7, child 2Link8, origin xyz=0 0 0.5 rpy=0 0 0, axis 1 1 0, limit lower=-3.14159 upper=3.14159 effort=0.0 velocity=0.0
- added joint 5Link0_5Link1: type revolute, parent 5Link0, child 5Link1, origin xyz=0 0.5 0 rpy=0 0 0, axis 1 1 0, limit lower=-3.14159 upper=3.14159 effort=0.0 velocity=0.0
- added joint 5Link1_5Link2: type revolute, parent 5Link1, child 5Link2, origin xyz=0 0.5 0 rpy=0 0 0, axis 1 1 0, limit lower=-3.14159 upper=3.14159 effort=0.0 velocity=0.0
- added joint 5Link2_5Link3: type revolute, parent 5Link2, child 5Link3, origin xyz=0 0.5 0 rpy=0 0 0, axis 1 1 0, limit lower=-3.14159 upper=3.14159 effort=0.0 velocity=0.0
- added joint 5Link3_5Link4: type revolute, parent 5Link3, child 5Link4, origin xyz=0 0.5 0 rpy=0 0 0, axis 1 1 0, limit lower=-3.14159 upper=3.14159 effort=0.0 velocity=0.0
- added joint 5Link4_5Link5: type revolute, parent 5Link4, child 5Link5, origin xyz=0 0.5 0 rpy=0 0 0, axis 1 1 0, limit lower=-3.14159 upper=3.14159 effort=0.0 velocity=0.0
- added joint 5Link5_5Link6: type revolute, parent 5Link5, child 5Link6, origin xyz=0 0.5 0 rpy=0 0 0, axis 1 1 0, limit lower=-3.14159 upper=3.14159 effort=0.0 velocity=0.0
- added joint 5Link6_5Link7: type revolute, parent 5Link6, child 5Link7, origin xyz=0 0.5 0 rpy=0 0 0, axis 1 1 0, limit lower=-3.14159 upper=3.14159 effort=0.0 velocity=0.0
- added joint 5Link7_5Link8: type revolute, parent 5Link7, child 5Link8, origin xyz=0 0.5 0 rpy=0 0 0, axis 1 1 0, limit lower=-3.14159 upper=3.14159 effort=0.0 velocity=0.0
- added joint 5Link8_5Link9: type revolute, parent 5Link8, child 5Link9, origin xyz=0 0.5 0 rpy=0 0 0, axis 1 1 0, limit lower=-3.14159 upper=3.14159 effort=0.0 velocity=0.0
- added joint 5Link9_5Link10: type revolute, parent 5Link9, child 5Link10, origin xyz=0 0.5 0 rpy=0 0 0, axis 1 1 0, limit lower=-3.14159 upper=3.14159 effort=0.0 velocity=0.0
- added joint Torso_5Link0: type revolute, parent Torso, child 5Link0, origin xyz=0.0 2.5 10.0 rpy=0 0 0, axis 1 1 0, limit lower=-3.14159 upper=3.14159 effort=0.0 velocity=0.0
