Commit message: etc

File: body.urdf (robot description, URDF)
Before this commit: robot robot, 64 links, 63 joints
Links:
- removed link 0Link10
- removed link 0Link9
- removed link 1Link10
- removed link 1Link11
- removed link 1Link8
- removed link 1Link9
- removed link 5Link10
- removed link 5Link8
- removed link 5Link9
- added link 4Link10, mass 1; collision box size=0.026448846593173037 0.03928793666944441 0.24893311354141412; visual box size=0.026448846593173037 0.03928793666944441 0.24893311354141412
- added link 4Link11, mass 1; collision box size=0.012797426045041305 0.7525783526559172 0.8832495799291901; visual box size=0.012797426045041305 0.7525783526559172 0.8832495799291901
- link 0Link0: geometry collision box size=0.08147499395085145 0.14054047989277973 0.6191209565049083; visual box size=0.08147499395085145 0.14054047989277973 0.6191209565049083
- link 0Link1: geometry collision box size=0.5123298203043289 0.3693593424343721 0.6796013670846055; visual box size=0.5123298203043289 0.3693593424343721 0.6796013670846055
- link 0Link2: geometry collision box size=0.3113693380974061 0.44398465136514054 0.9786921865412567; visual box size=0.3113693380974061 0.44398465136514054 0.9786921865412567
- link 0Link3: geometry collision box size=0.20107930147241082 0.3504573838961985 0.7385122247105147; visual box size=0.20107930147241082 0.3504573838961985 0.7385122247105147
- link 0Link4: geometry collision box size=0.7628706667154271 0.9013277680984515 0.622928951038159; visual box size=0.7628706667154271 0.9013277680984515 0.622928951038159
- link 0Link5: geometry collision box size=0.4360131964764571 0.1411226223086387 0.8643535029572721; visual box size=0.4360131964764571 0.1411226223086387 0.8643535029572721
- link 0Link6: geometry collision box size=0.23643916845403712 0.19055146283388313 0.8588389609174538; visual box size=0.23643916845403712 0.19055146283388313 0.8588389609174538
- link 0Link7: geometry collision box size=0.7120390431599731 0.2241763157095089 0.07837687327816412; visual box size=0.7120390431599731 0.2241763157095089 0.07837687327816412
- link 0Link8: geometry collision box size=0.6452625580272596 0.21732208381757523 0.3952490436212399; visual box size=0.6452625580272596 0.21732208381757523 0.3952490436212399
- link 1Link0: geometry collision box size=0.5611064218265784 0.023738996595601525 0.2773455997806866; visual box size=0.5611064218265784 0.023738996595601525 0.2773455997806866
- link 1Link1: geometry collision box size=0.21912968586341064 0.8762187046055043 0.9027267428188421; visual box size=0.21912968586341064 0.8762187046055043 0.9027267428188421
- link 1Link2: geometry collision box size=0.03573759689516276 0.4508427680264927 0.8117511976595431; visual box size=0.03573759689516276 0.4508427680264927 0.8117511976595431
- link 1Link3: geometry collision box size=0.9861928531061597 0.6711130188366582 0.20047262693071433; visual box size=0.9861928531061597 0.6711130188366582 0.20047262693071433
- link 1Link4: geometry collision box size=0.1608489679731534 0.5270493998099223 0.4581914773550987; visual box size=0.1608489679731534 0.5270493998099223 0.4581914773550987
- link 1Link5: geometry collision box size=0.8788443631790409 0.3634838470812002 0.42513088366146445; visual box size=0.8788443631790409 0.3634838470812002 0.42513088366146445
- link 1Link6: geometry collision box size=0.152374821478234 0.10217061185443421 0.6433208607889155; visual box size=0.152374821478234 0.10217061185443421 0.6433208607889155
- link 1Link7: geometry collision box size=0.3751270494061114 0.08886378753798685 0.5008337680455894; visual box size=0.3751270494061114 0.08886378753798685 0.5008337680455894
- link 2Link0: geometry collision box size=0.031204886434937462 0.25078152856998415 0.8254222886536212; visual box size=0.031204886434937462 0.25078152856998415 0.8254222886536212
- link 2Link1: geometry collision box size=0.32784498805412077 0.7626969762006773 0.5615780423246785; visual box size=0.32784498805412077 0.7626969762006773 0.5615780423246785
- link 2Link2: geometry collision box size=0.21253130746710291 0.7772606183828451 0.7182823993475749; visual box size=0.21253130746710291 0.7772606183828451 0.7182823993475749
- link 2Link3: geometry collision box size=0.13168909224077285 0.4546547241401445 0.5922036364446855; visual box size=0.13168909224077285 0.4546547241401445 0.5922036364446855
- link 2Link4: geometry collision box size=0.05951409894605009 0.8143876570274232 0.9279909886526375; visual box size=0.05951409894605009 0.8143876570274232 0.9279909886526375
- link 2Link5: geometry collision box size=0.037763752543705564 0.4555210907508397 0.11781190387917295; visual box size=0.037763752543705564 0.4555210907508397 0.11781190387917295
- link 2Link6: geometry collision box size=0.41662244441596097 0.5693008320504263 0.34638963508253107; visual box size=0.41662244441596097 0.5693008320504263 0.34638963508253107
- link 2Link7: geometry collision box size=0.8748432677771076 0.74632414563396 0.5663299543751381; visual box size=0.8748432677771076 0.74632414563396 0.5663299543751381
- link 2Link8: geometry collision box size=0.4858905703950376 0.7331451257316202 0.3724756964362186; visual box size=0.4858905703950376 0.7331451257316202 0.3724756964362186
- link 3Link0: geometry collision box size=0.511614263813101 0.9756193226078377 0.29092031362693627; visual box size=0.511614263813101 0.9756193226078377 0.29092031362693627
- link 3Link1: geometry collision box size=0.022024117772981078 0.7088609722069521 0.7914074360856974; visual box size=0.022024117772981078 0.7088609722069521 0.7914074360856974
- link 3Link2: geometry collision box size=0.5794020950506692 0.8739738554601422 0.36214136524138174; visual box size=0.5794020950506692 0.8739738554601422 0.36214136524138174
- link 3Link3: geometry collision box size=0.5771083259420727 0.4447419065741829 0.7194812725038747; visual box size=0.5771083259420727 0.4447419065741829 0.7194812725038747
- link 3Link4: geometry collision box size=0.21266124972093114 0.22784293890574703 0.14960614116396098; visual box size=0.21266124972093114 0.22784293890574703 0.14960614116396098
- link 3Link5: geometry collision box size=0.3001235031650613 0.05219311942129423 0.6079760767918807; visual box size=0.3001235031650613 0.05219311942129423 0.6079760767918807
- link 3Link6: geometry collision box size=0.5893312147712936 0.42755990803583643 0.14288053709602133; visual box size=0.5893312147712936 0.42755990803583643 0.14288053709602133
- link 3Link7: geometry collision box size=0.09698311225700318 0.8792425851813984 0.06517116863581418; visual box size=0.09698311225700318 0.8792425851813984 0.06517116863581418
- link 3Link8: geometry collision box size=0.9104490458841785 0.020602886451667413 0.42278429919678817; visual box size=0.9104490458841785 0.020602886451667413 0.42278429919678817
- link 3Link9: geometry collision box size=0.1900006541580418 0.4973406165333196 0.038375498775969796; visual box size=0.1900006541580418 0.4973406165333196 0.038375498775969796
- link 4Link0: geometry collision box size=0.2559209851906844 0.07799988220206522 0.6088175372554291; visual box size=0.2559209851906844 0.07799988220206522 0.6088175372554291
- link 4Link1: geometry collision box size=0.9102382886316495 0.608384782277814 0.5506850816800486; visual box size=0.9102382886316495 0.608384782277814 0.5506850816800486
- link 4Link2: geometry collision box size=0.14577246040170022 0.5654842287283828 0.004502496369882092; visual box size=0.14577246040170022 0.5654842287283828 0.004502496369882092
- link 4Link3: geometry collision box size=0.6271027849052255 0.4116057894980253 0.4948289626961808; visual box size=0.6271027849052255 0.4116057894980253 0.4948289626961808
- link 4Link4: geometry collision box size=0.15289733433760933 0.9797047454805201 0.015436215503958128; visual box size=0.15289733433760933 0.9797047454805201 0.015436215503958128
- link 4Link5: geometry collision box size=0.07200902609065973 0.4126601924847557 0.7176207972514611; visual box size=0.07200902609065973 0.4126601924847557 0.7176207972514611
- link 4Link6: geometry collision box size=0.21774563191531737 0.2549217986415636 0.10309226655570214; visual box size=0.21774563191531737 0.2549217986415636 0.10309226655570214
- link 4Link7: geometry collision box size=0.8444522768453772 0.05266904152898921 0.12364528319195478; visual box size=0.8444522768453772 0.05266904152898921 0.12364528319195478
- link 4Link8: geometry collision box size=0.33879923027612335 0.5253209570385338 0.27494438472318405; visual box size=0.33879923027612335 0.5253209570385338 0.27494438472318405
- link 4Link9: geometry collision box size=0.1437304799524648 0.431682374346959 0.0055109772435726345; visual box size=0.1437304799524648 0.431682374346959 0.0055109772435726345
- link 5Link0: geometry collision box size=0.5562705751460084 0.9469825465717662 0.8235551157571327; visual box size=0.5562705751460084 0.9469825465717662 0.8235551157571327
- link 5Link1: geometry collision box size=0.6117951925197312 0.6784412454164851 0.7459367521201818; visual box size=0.6117951925197312 0.6784412454164851 0.7459367521201818
- link 5Link2: geometry collision box size=0.3666774298218336 0.43705821020608926 0.6532834251628996; visual box size=0.3666774298218336 0.43705821020608926 0.6532834251628996
- link 5Link3: geometry collision box size=0.9581739461286448 0.43235225556642753 0.27186252457170634; visual box size=0.9581739461286448 0.43235225556642753 0.27186252457170634
- link 5Link4: geometry collision box size=0.41761860457048505 0.3797101314054786 0.3126991717122729; visual box size=0.41761860457048505 0.3797101314054786 0.3126991717122729
- link 5Link5: geometry collision box size=0.5997015443912238 0.8472014270932673 0.36138491430635844; visual box size=0.5997015443912238 0.8472014270932673 0.36138491430635844
- link 5Link6: geometry collision box size=0.8539650992882376 0.5034683588669182 0.7320340817247725; visual box size=0.8539650992882376 0.5034683588669182 0.7320340817247725
- link 5Link7: geometry collision box size=0.664564482332659 0.5355319795177523 0.31128331878972704; visual box size=0.664564482332659 0.5355319795177523 0.31128331878972704
Joints:
- removed joint 0Link8_0Link9
- removed joint 0Link9_0Link10
- removed joint 1Link10_1Link11
- removed joint 1Link7_1Link8
- removed joint 1Link8_1Link9
- removed joint 1Link9_1Link10
- removed joint 5Link7_5Link8
- removed joint 5Link8_5Link9
- removed joint 5Link9_5Link10
- added joint 4Link10_4Link11: type revolute, parent 4Link10, child 4Link11, origin xyz=0 -0.5 0 rpy=0 0 0, axis 1 1 0, limit lower=-3.14159 upper=3.14159 effort=0.0 velocity=0.0
- added joint 4Link9_4Link10: type revolute, parent 4Link9, child 4Link10, origin xyz=0 -0.5 0 rpy=0 0 0, axis 1 1 0, limit lower=-3.14159 upper=3.14159 effort=0.0 velocity=0.0

Commit message: etc

File: body.urdf (robot description, URDF)
Before this commit: robot robot, 64 links, 63 joints
Links:
- removed link 0Link10
- removed link 1Link10
- removed link 1Link11
- removed link 1Link8
- removed link 1Link9
- removed link 3Link8
- removed link 3Link9
- removed link 4Link0
- removed link 4Link1
- removed link 4Link2
- removed link 4Link3
- removed link 4Link4
- removed link 4Link5
- removed link 4Link6
- removed link 4Link7
- removed link 4Link8
- removed link 4Link9
- removed link 5Link0
- removed link 5Link1
- removed link 5Link10
- removed link 5Link2
- removed link 5Link3
- removed link 5Link4
- removed link 5Link5
- removed link 5Link6
- removed link 5Link7
- removed link 5Link8
- removed link 5Link9
- added link 2Link10, mass 1; collision box size=0.43604596471626267 0.6944947390068101 0.2218371709329312; visual box size=0.43604596471626267 0.6944947390068101 0.2218371709329312
- added link 2Link11, mass 1; collision box size=0.3738801982105847 0.5766578621332 0.49321567677687017; visual box size=0.3738801982105847 0.5766578621332 0.49321567677687017
- added link 2Link9, mass 1; collision box size=0.16406329004772158 0.0645627962595331 0.2799817264920542; visual box size=0.16406329004772158 0.0645627962595331 0.2799817264920542
- link 0Link0: geometry collision box size=0.6799388111058238 0.5344085950529291 0.3720070180127689; visual box size=0.6799388111058238 0.5344085950529291 0.3720070180127689
- link 0Link1: geometry collision box size=0.769388328990518 0.373257026250578 0.09209990874263252; visual box size=0.769388328990518 0.373257026250578 0.09209990874263252
- link 0Link2: geometry collision box size=0.9082874948578392 0.0735760606871273 0.984464306423496; visual box size=0.9082874948578392 0.0735760606871273 0.984464306423496
- link 0Link3: geometry collision box size=0.9404060231699861 0.7642645322711037 0.29471219626464973; visual box size=0.9404060231699861 0.7642645322711037 0.29471219626464973
- link 0Link4: geometry collision box size=0.9007653272550815 0.4091055077018383 0.3955914963797865; visual box size=0.9007653272550815 0.4091055077018383 0.3955914963797865
- link 0Link5: geometry collision box size=0.8575511101954564 0.6100695739805885 0.4546487579953742; visual box size=0.8575511101954564 0.6100695739805885 0.4546487579953742
- link 0Link6: geometry collision box size=0.0890067546003499 0.05485425115740472 0.0950830826371386; visual box size=0.0890067546003499 0.05485425115740472 0.0950830826371386
- link 0Link7: geometry collision box size=0.7479833741127472 0.2598744732392907 0.29635905137236485; visual box size=0.7479833741127472 0.2598744732392907 0.29635905137236485
- link 0Link8: geometry collision box size=0.21780658306231826 0.0032966136014966896 0.7407283595439385; visual box size=0.21780658306231826 0.0032966136014966896 0.7407283595439385
- link 0Link9: geometry collision box size=0.18213315021756882 0.13513897398413643 0.1965315440105445; visual box size=0.18213315021756882 0.13513897398413643 0.1965315440105445
- link 1Link0: geometry collision box size=0.08051835978755939 0.2390070752327731 0.6859216182815692; visual box size=0.08051835978755939 0.2390070752327731 0.6859216182815692
- link 1Link1: geometry collision box size=0.3261678554427939 0.4018298356358374 0.5441828355776668; visual box size=0.3261678554427939 0.4018298356358374 0.5441828355776668
- link 1Link2: geometry collision box size=0.048469142961951484 0.7974239187293982 0.26575432969954915; visual box size=0.048469142961951484 0.7974239187293982 0.26575432969954915
- link 1Link3: geometry collision box size=0.4356749069684569 0.17103606942936878 0.2891145704716451; visual box size=0.4356749069684569 0.17103606942936878 0.2891145704716451
- link 1Link4: geometry collision box size=0.135162412082513 0.47300338764126026 0.44307763576371806; visual box size=0.135162412082513 0.47300338764126026 0.44307763576371806
- link 1Link5: geometry collision box size=0.9255513321230829 0.19941891445943372 0.9564510180070154; visual box size=0.9255513321230829 0.19941891445943372 0.9564510180070154
- link 1Link6: geometry collision box size=0.4840745339509802 0.2019439345025026 0.3742460819261223; visual box size=0.4840745339509802 0.2019439345025026 0.3742460819261223
- link 1Link7: geometry collision box size=0.9904859577410241 0.23373254613873073 0.7277021773313438; visual box size=0.9904859577410241 0.23373254613873073 0.7277021773313438
- link 2Link0: geometry collision box size=0.6559417399480069 0.3335276738611145 0.1234919042744611; visual box size=0.6559417399480069 0.3335276738611145 0.1234919042744611
- link 2Link1: geometry collision box size=0.7168843875030104 0.13764100506164056 0.033357250121881954; visual box size=0.7168843875030104 0.13764100506164056 0.033357250121881954
- link 2Link2: geometry collision box size=0.4516752986928182 0.33960953600942956 0.3616195591300625; visual box size=0.4516752986928182 0.33960953600942956 0.3616195591300625
- link 2Link3: geometry collision box size=0.2846756579023684 0.6378333419240165 0.45995465021578585; visual box size=0.2846756579023684 0.6378333419240165 0.45995465021578585
- link 2Link4: geometry collision box size=0.44726149272296356 0.7640716536234862 0.15829962372158557; visual box size=0.44726149272296356 0.7640716536234862 0.15829962372158557
- link 2Link5: geometry collision box size=0.3093651927015797 0.9553857879488363 0.3107944309223495; visual box size=0.3093651927015797 0.9553857879488363 0.3107944309223495
- link 2Link6: geometry collision box size=0.09291424646698465 0.06744703204703495 0.5335621232230046; visual box size=0.09291424646698465 0.06744703204703495 0.5335621232230046
- link 2Link7: geometry collision box size=0.5124112921541237 0.6051678561496113 0.3128419347769522; visual box size=0.5124112921541237 0.6051678561496113 0.3128419347769522
- link 2Link8: geometry collision box size=0.572499862474388 0.38216583292901185 0.22908790101568344; visual box size=0.572499862474388 0.38216583292901185 0.22908790101568344
- link 3Link0: geometry collision box size=0.6471451741296697 0.42377949754624566 0.6810574793765525; visual box size=0.6471451741296697 0.42377949754624566 0.6810574793765525
- link 3Link1: geometry collision box size=0.2256824761438596 0.8175320928091465 0.09398875242352867; visual box size=0.2256824761438596 0.8175320928091465 0.09398875242352867
- link 3Link2: geometry collision box size=0.4997655825357854 0.44866672402321006 0.2790738847689026; visual box size=0.4997655825357854 0.44866672402321006 0.2790738847689026
- link 3Link3: geometry collision box size=0.8802808693619764 0.019000121741561182 0.3052442566203777; visual box size=0.8802808693619764 0.019000121741561182 0.3052442566203777
- link 3Link4: geometry collision box size=0.9337805562734951 0.08725982271783694 0.20426276503148832; visual box size=0.9337805562734951 0.08725982271783694 0.20426276503148832
- link 3Link5: geometry collision box size=0.7771508207623304 0.7251025870327032 0.21723625064253382; visual box size=0.7771508207623304 0.7251025870327032 0.21723625064253382
- link 3Link6: geometry collision box size=0.8061593324257237 0.2187322741678429 0.2525261938481642; visual box size=0.8061593324257237 0.2187322741678429 0.2525261938481642
- link 3Link7: geometry collision box size=0.7543899136086529 0.16227847063603118 0.7648319400132971; visual box size=0.7543899136086529 0.16227847063603118 0.7648319400132971
Joints:
- removed joint 0Link9_0Link10
- removed joint 1Link10_1Link11
- removed joint 1Link7_1Link8
- removed joint 1Link8_1Link9
- removed joint 1Link9_1Link10
- removed joint 3Link7_3Link8
- removed joint 3Link8_3Link9
- removed joint 4Link0_4Link1
- removed joint 4Link1_4Link2
- removed joint 4Link2_4Link3
- removed joint 4Link3_4Link4
- removed joint 4Link4_4Link5
- removed joint 4Link5_4Link6
- removed joint 4Link6_4Link7
- removed joint 4Link7_4Link8
- removed joint 4Link8_4Link9
- removed joint 5Link0_5Link1
- removed joint 5Link1_5Link2
- removed joint 5Link2_5Link3
- removed joint 5Link3_5Link4
- removed joint 5Link4_5Link5
- removed joint 5Link5_5Link6
- removed joint 5Link6_5Link7
- removed joint 5Link7_5Link8
- removed joint 5Link8_5Link9
- removed joint 5Link9_5Link10
- removed joint Torso_4Link0
- removed joint Torso_5Link0
- added joint 2Link10_2Link11: type revolute, parent 2Link10, child 2Link11, origin xyz=0 0 0.5 rpy=0 0 0, axis 1 1 0, limit lower=-3.14159 upper=3.14159 effort=0.0 velocity=0.0
- added joint 2Link8_2Link9: type revolute, parent 2Link8, child 2Link9, origin xyz=0 0 0.5 rpy=0 0 0, axis 1 1 0, limit lower=-3.14159 upper=3.14159 effort=0.0 velocity=0.0
- added joint 2Link9_2Link10: type revolute, parent 2Link9, child 2Link10, origin xyz=0 0 0.5 rpy=0 0 0, axis 1 1 0, limit lower=-3.14159 upper=3.14159 effort=0.0 velocity=0.0
