Commit message: etc

File: body.urdf (robot description, URDF)
Before this commit: robot robot, 39 links, 38 joints
Links:
- added link 0Link10, mass 1; collision box size=0.15629635637716488 0.06784355195729397 0.16654174878801575; visual box size=0.15629635637716488 0.06784355195729397 0.16654174878801575
- added link 0Link11, mass 1; collision box size=0.2301322302544988 0.7211286907999914 0.618042574081211; visual box size=0.2301322302544988 0.7211286907999914 0.618042574081211
- added link 0Link12, mass 1; collision box size=0.9566610826822173 0.7003009325986544 0.5358773636590153; visual box size=0.9566610826822173 0.7003009325986544 0.5358773636590153
- added link 0Link13, mass 1; collision box size=0.2647853339593573 0.6048753489914247 0.30284738073346484; visual box size=0.2647853339593573 0.6048753489914247 0.30284738073346484
- added link 0Link14, mass 1; collision box size=0.04705018607613498 0.41805156645969765 0.5275875957564469; visual box size=0.04705018607613498 0.41805156645969765 0.5275875957564469
- added link 0Link15, mass 1; collision box size=0.1512919248503144 0.33344561706960596 0.6610549306428979; visual box size=0.1512919248503144 0.33344561706960596 0.6610549306428979
- added link 0Link16, mass 1; collision box size=0.12413599875686221 0.9711510185430606 0.3580913729420746; visual box size=0.12413599875686221 0.9711510185430606 0.3580913729420746
- added link 1Link10, mass 1; collision box size=0.9780254262240613 0.8620866614665242 0.8439109155060915; visual box size=0.9780254262240613 0.8620866614665242 0.8439109155060915
- added link 1Link11, mass 1; collision box size=0.19586086534238834 0.4676502110614217 0.9146416067377156; visual box size=0.19586086534238834 0.4676502110614217 0.9146416067377156
- added link 1Link12, mass 1; collision box size=0.37966643711310655 0.04397798293005728 0.2228535333009578; visual box size=0.37966643711310655 0.04397798293005728 0.2228535333009578
- added link 1Link13, mass 1; collision box size=0.37839274928103817 0.8623292639440193 0.8244462882156565; visual box size=0.37839274928103817 0.8623292639440193 0.8244462882156565
- added link 1Link8, mass 1; collision box size=0.1185437145253565 0.45264249620780517 0.35835697807230404; visual box size=0.1185437145253565 0.45264249620780517 0.35835697807230404
- added link 1Link9, mass 1; collision box size=0.034108152849768425 0.24520433958940935 0.269728415292645; visual box size=0.034108152849768425 0.24520433958940935 0.269728415292645
- added link 2Link12, mass 1; collision box size=0.0029504597259258913 0.006212689504316082 0.12808952721842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; visual box size=0.0029504597259258913 0.006212689504316082 0.12808952721842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
- added link 2Link13, mass 1; collision box size=0.5782443255497006 0.4047548078622113 0.6616355604177938; visual box size=0.5782443255497006 0.4047548078622113 0.6616355604177938
- added link 2Link14, mass 1; collision box size=0.441025021112498 0.40184004684415386 0.4214990741486232; visual box size=0.441025021112498 0.40184004684415386 0.4214990741486232
- added link 2Link15, mass 1; collision box size=0.21901947997240112 0.5220825843197493 0.5784310791025122; visual box size=0.21901947997240112 0.5220825843197493 0.5784310791025122
- added link 3Link10, mass 1; collision box size=0.6646910058629291 0.6660451581848106 0.3826266697623675; visual box size=0.6646910058629291 0.6660451581848106 0.3826266697623675
- added link 3Link11, mass 1; collision box size=0.7444540809610773 0.864205896893844 0.26536569607675864; visual box size=0.7444540809610773 0.864205896893844 0.26536569607675864
- added link 3Link12, mass 1; collision box size=0.3763081958131895 0.912073069739509 0.18602088725891486; visual box size=0.3763081958131895 0.912073069739509 0.18602088725891486
- added link 3Link13, mass 1; collision box size=0.3775661463236948 0.42495167921644506 0.9044150373712919; visual box size=0.3775661463236948 0.42495167921644506 0.9044150373712919
- added link 3Link8, mass 1; collision box size=0.8780860999148932 0.7035154160620073 0.21090226321522398; visual box size=0.8780860999148932 0.7035154160620073 0.21090226321522398
- added link 3Link9, mass 1; collision box size=0.2512969004498866 0.9808390304789087 0.2794385627371576; visual box size=0.2512969004498866 0.9808390304789087 0.2794385627371576
- link 0Link0: geometry collision box size=0.9526084856470317 0.857823789220692 0.9109969765779635; visual box size=0.9526084856470317 0.857823789220692 0.9109969765779635
- link 0Link1: geometry collision box size=0.5702651225969384 0.2969190194551019 0.3209942926973711; visual box size=0.5702651225969384 0.2969190194551019 0.3209942926973711
- link 0Link2: geometry collision box size=0.9561647977753285 0.40102610761719315 0.5918012709038877; visual box size=0.9561647977753285 0.40102610761719315 0.5918012709038877
- link 0Link3: geometry collision box size=0.007925722802325508 0.04927765919278437 0.7524821349549202; visual box size=0.007925722802325508 0.04927765919278437 0.7524821349549202
- link 0Link4: geometry collision box size=0.5029987335840149 0.6839465273442776 0.6719478653798212; visual box size=0.5029987335840149 0.6839465273442776 0.6719478653798212
- link 0Link5: geometry collision box size=0.09495811390634612 0.702045296932598 0.015636059049412232; visual box size=0.09495811390634612 0.702045296932598 0.015636059049412232
- link 0Link6: geometry collision box size=0.4662680732016795 0.4237880458058878 0.35775744447962843; visual box size=0.4662680732016795 0.4237880458058878 0.35775744447962843
- link 0Link7: geometry collision box size=0.07577637993617847 0.6117621938385724 0.12841411752476428; visual box size=0.07577637993617847 0.6117621938385724 0.12841411752476428
- link 0Link8: geometry collision box size=0.09355773874230289 0.30268635494142815 0.07831788699152964; visual box size=0.09355773874230289 0.30268635494142815 0.07831788699152964
- link 0Link9: geometry collision box size=0.7187327876964006 0.09975169481593527 0.6533306808545373; visual box size=0.7187327876964006 0.09975169481593527 0.6533306808545373
- link 1Link0: geometry collision box size=0.2968610759151319 0.42684862921955047 0.9814308581461079; visual box size=0.2968610759151319 0.42684862921955047 0.9814308581461079
- link 1Link1: geometry collision box size=0.21961219163138557 0.7367811061451195 0.5311150222194219; visual box size=0.21961219163138557 0.7367811061451195 0.5311150222194219
- link 1Link2: geometry collision box size=0.5313915287942091 0.6936264271508602 0.1638603471704112; visual box size=0.5313915287942091 0.6936264271508602 0.1638603471704112
- link 1Link3: geometry collision box size=0.49760846149876203 0.04773639678385322 0.8150847144498399; visual box size=0.49760846149876203 0.04773639678385322 0.8150847144498399
- link 1Link4: geometry collision box size=0.558578564787194 0.4811244331584438 0.038409778687265694; visual box size=0.558578564787194 0.4811244331584438 0.038409778687265694
- link 1Link5: geometry collision box size=0.2397944505707491 0.5717932329935865 0.8512684908481534; visual box size=0.2397944505707491 0.5717932329935865 0.8512684908481534
- link 1Link6: geometry collision box size=0.018636885301514527 0.712663558945338 0.33969241290824803; visual box size=0.018636885301514527 0.712663558945338 0.33969241290824803
- link 1Link7: geometry collision box size=0.5567293264747872 0.680712297341224 0.5969863397432013; visual box size=0.5567293264747872 0.680712297341224 0.5969863397432013
- link 2Link0: geometry collision box size=0.2969205175594043 0.403355366280455 0.7944034766236732; visual box size=0.2969205175594043 0.403355366280455 0.7944034766236732
- link 2Link1: geometry collision box size=0.08944868005042605 0.6580178704806214 0.35613502058337676; visual box size=0.08944868005042605 0.6580178704806214 0.35613502058337676
- link 2Link10: geometry collision box size=0.8101459050570706 0.36884670380932494 0.9866056600964334; visual box size=0.8101459050570706 0.36884670380932494 0.9866056600964334
- link 2Link11: geometry collision box size=0.09261859599262479 0.6711801566041524 0.6361467906297125; visual box size=0.09261859599262479 0.6711801566041524 0.6361467906297125
- link 2Link2: geometry collision box size=0.31419928513285755 0.7232559699970147 0.9435412283247877; visual box size=0.31419928513285755 0.7232559699970147 0.9435412283247877
- link 2Link3: geometry collision box size=0.9727221180071263 0.3162529521237918 0.7352712183796052; visual box size=0.9727221180071263 0.3162529521237918 0.7352712183796052
- link 2Link4: geometry collision box size=0.4071636491006084 0.9201790373080202 0.5212929840568531; visual box size=0.4071636491006084 0.9201790373080202 0.5212929840568531
- link 2Link5: geometry collision box size=0.9446462346412294 0.009267758064406717 0.43746298899893665; visual box size=0.9446462346412294 0.009267758064406717 0.43746298899893665
- link 2Link6: geometry collision box size=0.4061860120665206 0.6378012671086278 0.06760472292880082; visual box size=0.4061860120665206 0.6378012671086278 0.06760472292880082
- link 2Link7: geometry collision box size=0.82042758202129 0.8189115046699748 0.501774532288598; visual box size=0.82042758202129 0.8189115046699748 0.501774532288598
- link 2Link8: geometry collision box size=0.06391262887232607 0.9525171683635443 0.22259012784128307; visual box size=0.06391262887232607 0.9525171683635443 0.22259012784128307
- link 2Link9: geometry collision box size=0.9161681255833678 0.5253461092144237 0.012666419713111665; visual box size=0.9161681255833678 0.5253461092144237 0.012666419713111665
- link 3Link0: geometry collision box size=0.9489574487139847 0.7048289511707101 0.5767517639665383; visual box size=0.9489574487139847 0.7048289511707101 0.5767517639665383
- link 3Link1: geometry collision box size=0.1240068720299018 0.7900319999552657 0.48065468689352353; visual box size=0.1240068720299018 0.7900319999552657 0.48065468689352353
- link 3Link2: geometry collision box size=0.8162156526326959 0.6583760856999763 0.8310459648076431; visual box size=0.8162156526326959 0.6583760856999763 0.8310459648076431
- link 3Link3: geometry collision box size=0.4487522352171278 0.08971520201981764 0.37833044586113207; visual box size=0.4487522352171278 0.08971520201981764 0.37833044586113207
- link 3Link4: geometry collision box size=0.18947453795776514 0.4543273650766876 0.07640551217627056; visual box size=0.18947453795776514 0.4543273650766876 0.07640551217627056
- link 3Link5: geometry collision box size=0.5589178534560917 0.031183112250963263 0.9068047170316332; visual box size=0.5589178534560917 0.031183112250963263 0.9068047170316332
- link 3Link6: geometry collision box size=0.12438054254669584 0.5228732939341357 0.7112032833974533; visual box size=0.12438054254669584 0.5228732939341357 0.7112032833974533
- link 3Link7: geometry collision box size=0.9480456924693806 0.4538234601813955 0.8891416785829686; visual box size=0.9480456924693806 0.4538234601813955 0.8891416785829686
Joints:
- added joint 0Link10_0Link11: type revolute, parent 0Link10, child 0Link11, origin xyz=0 0 -0.5 rpy=0 0 0, axis 1 1 0, limit lower=-3.14159 upper=3.14159 effort=0.0 velocity=0.0
- added joint 0Link11_0Link12: type revolute, parent 0Link11, child 0Link12, origin xyz=0 0 -0.5 rpy=0 0 0, axis 1 1 0, limit lower=-3.14159 upper=3.14159 effort=0.0 velocity=0.0
- added joint 0Link12_0Link13: type revolute, parent 0Link12, child 0Link13, origin xyz=0 0 -0.5 rpy=0 0 0, axis 1 1 0, limit lower=-3.14159 upper=3.14159 effort=0.0 velocity=0.0
- added joint 0Link13_0Link14: type revolute, parent 0Link13, child 0Link14, origin xyz=0 0 -0.5 rpy=0 0 0, axis 1 1 0, limit lower=-3.14159 upper=3.14159 effort=0.0 velocity=0.0
- added joint 0Link14_0Link15: type revolute, parent 0Link14, child 0Link15, origin xyz=0 0 -0.5 rpy=0 0 0, axis 1 1 0, limit lower=-3.14159 upper=3.14159 effort=0.0 velocity=0.0
- added joint 0Link15_0Link16: type revolute, parent 0Link15, child 0Link16, origin xyz=0 0 -0.5 rpy=0 0 0, axis 1 1 0, limit lower=-3.14159 upper=3.14159 effort=0.0 velocity=0.0
- added joint 0Link9_0Link10: type revolute, parent 0Link9, child 0Link10, origin xyz=0 0 -0.5 rpy=0 0 0, axis 1 1 0, limit lower=-3.14159 upper=3.14159 effort=0.0 velocity=0.0
- added joint 1Link10_1Link11: type revolute, parent 1Link10, child 1Link11, origin xyz=-0.5 0 0 rpy=0 0 0, axis 1 1 0, limit lower=-3.14159 upper=3.14159 effort=0.0 velocity=0.0
- added joint 1Link11_1Link12: type revolute, parent 1Link11, child 1Link12, origin xyz=-0.5 0 0 rpy=0 0 0, axis 1 1 0, limit lower=-3.14159 upper=3.14159 effort=0.0 velocity=0.0
- added joint 1Link12_1Link13: type revolute, parent 1Link12, child 1Link13, origin xyz=-0.5 0 0 rpy=0 0 0, axis 1 1 0, limit lower=-3.14159 upper=3.14159 effort=0.0 velocity=0.0
- added joint 1Link7_1Link8: type revolute, parent 1Link7, child 1Link8, origin xyz=-0.5 0 0 rpy=0 0 0, axis 1 1 0, limit lower=-3.14159 upper=3.14159 effort=0.0 velocity=0.0
- added joint 1Link8_1Link9: type revolute, parent 1Link8, child 1Link9, origin xyz=-0.5 0 0 rpy=0 0 0, axis 1 1 0, limit lower=-3.14159 upper=3.14159 effort=0.0 velocity=0.0
- added joint 1Link9_1Link10: type revolute, parent 1Link9, child 1Link10, origin xyz=-0.5 0 0 rpy=0 0 0, axis 1 1 0, limit lower=-3.14159 upper=3.14159 effort=0.0 velocity=0.0
- added joint 2Link11_2Link12: type revolute, parent 2Link11, child 2Link12, origin xyz=0 0 0.5 rpy=0 0 0, axis 1 1 0, limit lower=-3.14159 upper=3.14159 effort=0.0 velocity=0.0
- added joint 2Link12_2Link13: type revolute, parent 2Link12, child 2Link13, origin xyz=0 0 0.5 rpy=0 0 0, axis 1 1 0, limit lower=-3.14159 upper=3.14159 effort=0.0 velocity=0.0
- added joint 2Link13_2Link14: type revolute, parent 2Link13, child 2Link14, origin xyz=0 0 0.5 rpy=0 0 0, axis 1 1 0, limit lower=-3.14159 upper=3.14159 effort=0.0 velocity=0.0
- added joint 2Link14_2Link15: type revolute, parent 2Link14, child 2Link15, origin xyz=0 0 0.5 rpy=0 0 0, axis 1 1 0, limit lower=-3.14159 upper=3.14159 effort=0.0 velocity=0.0
- added joint 3Link10_3Link11: type revolute, parent 3Link10, child 3Link11, origin xyz=0.5 0 0 rpy=0 0 0, axis 1 1 0, limit lower=-3.14159 upper=3.14159 effort=0.0 velocity=0.0
- added joint 3Link11_3Link12: type revolute, parent 3Link11, child 3Link12, origin xyz=0.5 0 0 rpy=0 0 0, axis 1 1 0, limit lower=-3.14159 upper=3.14159 effort=0.0 velocity=0.0
- added joint 3Link12_3Link13: type revolute, parent 3Link12, child 3Link13, origin xyz=0.5 0 0 rpy=0 0 0, axis 1 1 0, limit lower=-3.14159 upper=3.14159 effort=0.0 velocity=0.0
- added joint 3Link7_3Link8: type revolute, parent 3Link7, child 3Link8, origin xyz=0.5 0 0 rpy=0 0 0, axis 1 1 0, limit lower=-3.14159 upper=3.14159 effort=0.0 velocity=0.0
- added joint 3Link8_3Link9: type revolute, parent 3Link8, child 3Link9, origin xyz=0.5 0 0 rpy=0 0 0, axis 1 1 0, limit lower=-3.14159 upper=3.14159 effort=0.0 velocity=0.0
- added joint 3Link9_3Link10: type revolute, parent 3Link9, child 3Link10, origin xyz=0.5 0 0 rpy=0 0 0, axis 1 1 0, limit lower=-3.14159 upper=3.14159 effort=0.0 velocity=0.0
