Commit message: etc

File: body.urdf (robot description, URDF)
Before this commit: robot robot, 62 links, 61 joints
Links:
- removed link 0Link16
- removed link 2Link15
- removed link 3Link12
- removed link 3Link13
- added link 1Link14, mass 1; collision box size=0.9239620304793491 0.6137975230628351 0.309011975239347; visual box size=0.9239620304793491 0.6137975230628351 0.309011975239347
- added link 1Link15, mass 1; collision box size=0.25713474870492403 0.7229097207912762 0.231724125903373; visual box size=0.25713474870492403 0.7229097207912762 0.231724125903373
- added link 1Link16, mass 1; collision box size=0.06771729621829337 0.7698237212387375 0.846173070573634; visual box size=0.06771729621829337 0.7698237212387375 0.846173070573634
- added link 4Link0, mass 1; collision box size=0.5546320147706982 0.7988282212140577 0.8401717725873136; visual box size=0.5546320147706982 0.7988282212140577 0.8401717725873136
- added link 4Link1, mass 1; collision box size=0.7144063046395054 0.7153460150274972 0.847008537669469; visual box size=0.7144063046395054 0.7153460150274972 0.847008537669469
- added link 4Link10, mass 1; collision box size=0.9073729131647907 0.9479838169146321 0.9172288036787847; visual box size=0.9073729131647907 0.9479838169146321 0.9172288036787847
- added link 4Link11, mass 1; collision box size=0.5717868306652141 0.7105870514312667 0.4901869364777155; visual box size=0.5717868306652141 0.7105870514312667 0.4901869364777155
- added link 4Link12, mass 1; collision box size=0.8598653416745344 0.21692838588309626 0.9722476731263776; visual box size=0.8598653416745344 0.21692838588309626 0.9722476731263776
- added link 4Link13, mass 1; collision box size=0.83324100238752 0.04788174278380419 0.5843150095333147; visual box size=0.83324100238752 0.04788174278380419 0.5843150095333147
- added link 4Link14, mass 1; collision box size=0.20150611922624118 0.10651700846540657 0.8014743654475591; visual box size=0.20150611922624118 0.10651700846540657 0.8014743654475591
- added link 4Link2, mass 1; collision box size=0.16450447829249815 0.8105321090079429 0.4973104116742093; visual box size=0.16450447829249815 0.8105321090079429 0.4973104116742093
- added link 4Link3, mass 1; collision box size=0.48759858911099063 0.2566257950442167 0.6832413155735241; visual box size=0.48759858911099063 0.2566257950442167 0.6832413155735241
- added link 4Link4, mass 1; collision box size=0.14300950929484046 0.12132746749193235 0.25254528540659615; visual box size=0.14300950929484046 0.12132746749193235 0.25254528540659615
- added link 4Link5, mass 1; collision box size=0.5794618487726487 0.7973324285076486 0.17060968607078242; visual box size=0.5794618487726487 0.7973324285076486 0.17060968607078242
- added link 4Link6, mass 1; collision box size=0.8734394050277405 0.15516902247075515 0.28811344419688356; visual box size=0.8734394050277405 0.15516902247075515 0.28811344419688356
- added link 4Link7, mass 1; collision box size=0.7213695781572327 0.46160702328044845 0.638605450130043; visual box size=0.7213695781572327 0.46160702328044845 0.638605450130043
- added link 4Link8, mass 1; collision box size=0.5242080626170896 0.9030279125384774 0.1945354480050825; visual box size=0.5242080626170896 0.9030279125384774 0.1945354480050825
- added link 4Link9, mass 1; collision box size=0.3906588020781828 0.4217322542195996 0.6284040869880482; visual box size=0.3906588020781828 0.4217322542195996 0.6284040869880482
- added link 5Link0, mass 1; collision box size=0.9432545378701424 0.19502403612990282 0.035569040259760154; visual box size=0.9432545378701424 0.19502403612990282 0.035569040259760154
- added link 5Link1, mass 1; collision box size=0.01761286813994245 0.6454512880037108 0.7917352413515613; visual box size=0.01761286813994245 0.6454512880037108 0.7917352413515613
- added link 5Link10, mass 1; collision box size=0.7885440533438987 0.6898925920599798 0.964444804704827; visual box size=0.7885440533438987 0.6898925920599798 0.964444804704827
- added link 5Link11, mass 1; collision box size=0.2116415592830011 0.5552579405059801 0.8641740590532155; visual box size=0.2116415592830011 0.5552579405059801 0.8641740590532155
- added link 5Link12, mass 1; collision box size=0.9115341324819357 0.8595953062410175 0.8022726361328106; visual box size=0.9115341324819357 0.8595953062410175 0.8022726361328106
- added link 5Link13, mass 1; collision box size=0.4718003332761421 0.18537589335240667 0.8192249100453248; visual box size=0.4718003332761421 0.18537589335240667 0.8192249100453248
- added link 5Link14, mass 1; collision box size=0.022023940780812934 0.15059132272421882 0.9647971213736704; visual box size=0.022023940780812934 0.15059132272421882 0.9647971213736704
- added link 5Link15, mass 1; collision box size=0.17077498462405216 0.6842624519456902 0.9888201178433275; visual box size=0.17077498462405216 0.6842624519456902 0.9888201178433275
- added link 5Link16, mass 1; collision box size=0.6338337719111334 0.10503687200587597 0.2246999587737678; visual box size=0.6338337719111334 0.10503687200587597 0.2246999587737678
- added link 5Link17, mass 1; collision box size=0.4768488596500293 0.8076989608384175 0.5193976648999146; visual box size=0.4768488596500293 0.8076989608384175 0.5193976648999146
- added link 5Link2, mass 1; collision box size=0.6370108464932013 0.9789482965390233 0.7300499115867228; visual box size=0.6370108464932013 0.9789482965390233 0.7300499115867228
- added link 5Link3, mass 1; collision box size=0.49318830295484906 0.005607551616104711 0.11635715977680727; visual box size=0.49318830295484906 0.005607551616104711 0.11635715977680727
- added link 5Link4, mass 1; collision box size=0.3341565530448919 0.8568732135446673 0.4123486217132899; visual box size=0.3341565530448919 0.8568732135446673 0.4123486217132899
- added link 5Link5, mass 1; collision box size=0.4970174396873118 0.4947721608541188 0.8328122102869542; visual box size=0.4970174396873118 0.4947721608541188 0.8328122102869542
- added link 5Link6, mass 1; collision box size=0.5949200019909084 0.14322267539614908 0.6173610858338107; visual box size=0.5949200019909084 0.14322267539614908 0.6173610858338107
- added link 5Link7, mass 1; collision box size=0.23066188011616784 0.30781370091428706 0.12756525037104272; visual box size=0.23066188011616784 0.30781370091428706 0.12756525037104272
- added link 5Link8, mass 1; collision box size=0.7706670183613656 0.581517634745842 0.7824664758542763; visual box size=0.7706670183613656 0.581517634745842 0.7824664758542763
- added link 5Link9, mass 1; collision box size=0.2022414330749842 0.37501433815576213 0.13151543406963273; visual box size=0.2022414330749842 0.37501433815576213 0.13151543406963273
- link 0Link0: geometry collision box size=0.8221342255418969 0.9791990067224007 0.6906269718285101; visual box size=0.8221342255418969 0.9791990067224007 0.6906269718285101
- link 0Link1: geometry collision box size=0.9099559170834326 0.06531179369990181 0.14046321562566344; visual box size=0.9099559170834326 0.06531179369990181 0.14046321562566344
- link 0Link10: geometry collision box size=0.3713100138355059 0.3031238170846784 0.5877629930479419; visual box size=0.3713100138355059 0.3031238170846784 0.5877629930479419
- link 0Link11: geometry collision box size=0.23977468541604308 0.5183144147645248 0.7990595861911534; visual box size=0.23977468541604308 0.5183144147645248 0.7990595861911534
- link 0Link12: geometry collision box size=0.9099814039805647 0.5048351795900313 0.3021081600673502; visual box size=0.9099814039805647 0.5048351795900313 0.3021081600673502
- link 0Link13: geometry collision box size=0.9603946911581301 0.36268990001934553 0.3857568191557953; visual box size=0.9603946911581301 0.36268990001934553 0.3857568191557953
- link 0Link14: geometry collision box size=0.8295003478761205 0.9763828975602352 0.5380586555368676; visual box size=0.8295003478761205 0.9763828975602352 0.5380586555368676
- link 0Link15: geometry collision box size=0.6958595034455172 0.22470602912904547 0.37983326232924475; visual box size=0.6958595034455172 0.22470602912904547 0.37983326232924475
- link 0Link2: geometry collision box size=0.21001702000441247 0.5022771070248355 0.7285303930594861; visual box size=0.21001702000441247 0.5022771070248355 0.7285303930594861
- link 0Link3: geometry collision box size=0.8190482150245411 0.27462393959377485 0.22432420829600253; visual box size=0.8190482150245411 0.27462393959377485 0.22432420829600253
- link 0Link4: geometry collision box size=0.7695968681017931 0.5069975485685974 0.33951004835796705; visual box size=0.7695968681017931 0.5069975485685974 0.33951004835796705
- link 0Link5: geometry collision box size=0.0728495681088066 0.9584779962719604 0.0900211706984354; visual box size=0.0728495681088066 0.9584779962719604 0.0900211706984354
- link 0Link6: geometry collision box size=0.3630712509389298 0.2789142230797602 0.09091833770576807; visual box size=0.3630712509389298 0.2789142230797602 0.09091833770576807
- link 0Link7: geometry collision box size=0.6740971122417486 0.3146826257266945 0.15283341620026358; visual box size=0.6740971122417486 0.3146826257266945 0.15283341620026358
- link 0Link8: geometry collision box size=0.09683243327375168 0.6270001497093411 0.7736414808167961; visual box size=0.09683243327375168 0.6270001497093411 0.7736414808167961
- link 0Link9: geometry collision box size=0.24376627417662944 0.7841385961537998 0.6569570447731534; visual box size=0.24376627417662944 0.7841385961537998 0.6569570447731534
- link 1Link0: geometry collision box size=0.16410062455896746 0.28424492276888824 0.03817779994909121; visual box size=0.16410062455896746 0.28424492276888824 0.03817779994909121
- link 1Link1: geometry collision box size=0.8478519605480248 0.859396666216652 0.5916333958282819; visual box size=0.8478519605480248 0.859396666216652 0.5916333958282819
- link 1Link10: geometry collision box size=0.49691234267159967 0.3749924088071055 0.7996289629747447; visual box size=0.49691234267159967 0.3749924088071055 0.7996289629747447
- link 1Link11: geometry collision box size=0.6917932054331869 0.7917243568758577 0.9037654973437432; visual box size=0.6917932054331869 0.7917243568758577 0.9037654973437432
- link 1Link12: geometry collision box size=0.7592601416912467 0.8762225722366541 0.7753375670652515; visual box size=0.7592601416912467 0.8762225722366541 0.7753375670652515
- link 1Link13: geometry collision box size=0.024683184976927675 0.2609912114858809 0.28330591477217415; visual box size=0.024683184976927675 0.2609912114858809 0.28330591477217415
- link 1Link2: geometry collision box size=0.9826245307003062 0.9285944188688908 0.8032271937538122; visual box size=0.9826245307003062 0.9285944188688908 0.8032271937538122
- link 1Link3: geometry collision box size=0.5903365146368347 0.0710061383871019 0.7397206419707721; visual box size=0.5903365146368347 0.0710061383871019 0.7397206419707721
- link 1Link4: geometry collision box size=0.916328611500067 0.7556438098879499 0.3289725961948632; visual box size=0.916328611500067 0.7556438098879499 0.3289725961948632
- link 1Link5: geometry collision box size=0.1075820355010233 0.5105201222336114 0.06926056893769927; visual box size=0.1075820355010233 0.5105201222336114 0.06926056893769927
- link 1Link6: geometry collision box size=0.13048956190362992 0.9481275692426019 0.3535704363507991; visual box size=0.13048956190362992 0.9481275692426019 0.3535704363507991
- link 1Link7: geometry collision box size=0.12252829504017915 0.09534049603449324 0.4701427344504011; visual box size=0.12252829504017915 0.09534049603449324 0.4701427344504011
- link 1Link8: geometry collision box size=0.10449967097126112 0.7295839409772492 0.3807060237947667; visual box size=0.10449967097126112 0.7295839409772492 0.3807060237947667
- link 1Link9: geometry collision box size=0.6139201493514196 0.6420863400543745 0.3252336530555153; visual box size=0.6139201493514196 0.6420863400543745 0.3252336530555153
- link 2Link0: geometry collision box size=0.07121047489279853 0.32149125462199934 0.4739579996703943; visual box size=0.07121047489279853 0.32149125462199934 0.4739579996703943
- link 2Link1: geometry collision box size=0.8561720803131605 0.7200565747090011 0.5153335193962123; visual box size=0.8561720803131605 0.7200565747090011 0.5153335193962123
- link 2Link10: geometry collision box size=0.8718747655084217 0.7758627076710288 0.2552669322970982; visual box size=0.8718747655084217 0.7758627076710288 0.2552669322970982
- link 2Link11: geometry collision box size=0.02266549655706518 0.5394360733568543 0.4686286913148012; visual box size=0.02266549655706518 0.5394360733568543 0.4686286913148012
- link 2Link12: geometry collision box size=0.021078156489411137 0.42614867857055483 0.5371674851497672; visual box size=0.021078156489411137 0.42614867857055483 0.5371674851497672
- link 2Link13: geometry collision box size=0.2240397840358339 0.05842736457373787 0.4752755708158697; visual box size=0.2240397840358339 0.05842736457373787 0.4752755708158697
- link 2Link14: geometry collision box size=0.29155778187096426 0.5064901504085638 0.4763226226827114; visual box size=0.29155778187096426 0.5064901504085638 0.4763226226827114
- link 2Link2: geometry collision box size=0.5645282017145019 0.05837124238337554 0.4537131774020897; visual box size=0.5645282017145019 0.05837124238337554 0.4537131774020897
- link 2Link3: geometry collision box size=0.7828887947439889 0.49027478057470775 0.09470346112301031; visual box size=0.7828887947439889 0.49027478057470775 0.09470346112301031
- link 2Link4: geometry collision box size=0.38020316041837543 0.7020498842361892 0.9711598135011555; visual box size=0.38020316041837543 0.7020498842361892 0.9711598135011555
- link 2Link5: geometry collision box size=0.035163027816065284 0.5444123197586422 0.11710633585472074; visual box size=0.035163027816065284 0.5444123197586422 0.11710633585472074
- link 2Link6: geometry collision box size=0.9510569209422374 0.27661067257750305 0.44262053272057855; visual box size=0.9510569209422374 0.27661067257750305 0.44262053272057855
- link 2Link7: geometry collision box size=0.2004370069517437 0.783486644626277 0.5517764035509285; visual box size=0.2004370069517437 0.783486644626277 0.5517764035509285
- link 2Link8: geometry collision box size=0.12337201452190971 0.23290994048790525 0.7379961125615505; visual box size=0.12337201452190971 0.23290994048790525 0.7379961125615505
- link 2Link9: geometry collision box size=0.6809768267099374 0.9892915913898775 0.5628663967830445; visual box size=0.6809768267099374 0.9892915913898775 0.5628663967830445
- link 3Link0: geometry collision box size=0.3402759144541343 0.29955847697187543 0.22313960191943605; visual box size=0.3402759144541343 0.29955847697187543 0.22313960191943605
- link 3Link1: geometry collision box size=0.4034694710494544 0.8606736929605765 0.48525739625987463; visual box size=0.4034694710494544 0.8606736929605765 0.48525739625987463
- link 3Link10: geometry collision box size=0.13909878903331663 0.08415185742597353 0.10896682576440786; visual box size=0.13909878903331663 0.08415185742597353 0.10896682576440786
- link 3Link11: geometry collision box size=0.7567342759339747 0.6731741462721306 0.8972508256043713; visual box size=0.7567342759339747 0.6731741462721306 0.8972508256043713
- link 3Link2: geometry collision box size=0.218626960592762 0.18437429776514014 0.12781696601817505; visual box size=0.218626960592762 0.18437429776514014 0.12781696601817505
- link 3Link3: geometry collision box size=0.3779650468763174 0.9916814490290685 0.6825706965614641; visual box size=0.3779650468763174 0.9916814490290685 0.6825706965614641
- link 3Link4: geometry collision box size=0.5348824268008733 0.6834661852771728 0.20101009001996362; visual box size=0.5348824268008733 0.6834661852771728 0.20101009001996362
- link 3Link5: geometry collision box size=0.32188517577387876 0.677321052469209 0.381133202477799; visual box size=0.32188517577387876 0.677321052469209 0.381133202477799
- link 3Link6: geometry collision box size=0.7957340863038229 0.9598874763528398 0.28245574871080004; visual box size=0.7957340863038229 0.9598874763528398 0.28245574871080004
- link 3Link7: geometry collision box size=0.037424575038389474 0.32827795985687036 0.7641128344745499; visual box size=0.037424575038389474 0.32827795985687036 0.7641128344745499
- link 3Link8: geometry collision box size=0.41931780824728826 0.013096846056042333 0.8397626746271977; visual box size=0.41931780824728826 0.013096846056042333 0.8397626746271977
- link 3Link9: geometry collision box size=0.9491579217747715 0.8411016634648093 0.40337110134752996; visual box size=0.9491579217747715 0.8411016634648093 0.40337110134752996
Joints:
- removed joint 0Link15_0Link16
- removed joint 2Link14_2Link15
- removed joint 3Link11_3Link12
- removed joint 3Link12_3Link13
- added joint 1Link13_1Link14: type revolute, parent 1Link13, child 1Link14, origin xyz=-0.5 0 0 rpy=0 0 0, axis 1 1 0, limit lower=-3.14159 upper=3.14159 effort=0.0 velocity=0.0
- added joint 1Link14_1Link15: type revolute, parent 1Link14, child 1Link15, origin xyz=-0.5 0 0 rpy=0 0 0, axis 1 1 0, limit lower=-3.14159 upper=3.14159 effort=0.0 velocity=0.0
- added joint 1Link15_1Link16: type revolute, parent 1Link15, child 1Link16, origin xyz=-0.5 0 0 rpy=0 0 0, axis 1 1 0, limit lower=-3.14159 upper=3.14159 effort=0.0 velocity=0.0
- added joint 4Link0_4Link1: type revolute, parent 4Link0, child 4Link1, origin xyz=0 -0.5 0 rpy=0 0 0, axis 1 1 0, limit lower=-3.14159 upper=3.14159 effort=0.0 velocity=0.0
- added joint 4Link10_4Link11: type revolute, parent 4Link10, child 4Link11, origin xyz=0 -0.5 0 rpy=0 0 0, axis 1 1 0, limit lower=-3.14159 upper=3.14159 effort=0.0 velocity=0.0
- added joint 4Link11_4Link12: type revolute, parent 4Link11, child 4Link12, origin xyz=0 -0.5 0 rpy=0 0 0, axis 1 1 0, limit lower=-3.14159 upper=3.14159 effort=0.0 velocity=0.0
- added joint 4Link12_4Link13: type revolute, parent 4Link12, child 4Link13, origin xyz=0 -0.5 0 rpy=0 0 0, axis 1 1 0, limit lower=-3.14159 upper=3.14159 effort=0.0 velocity=0.0
- added joint 4Link13_4Link14: type revolute, parent 4Link13, child 4Link14, origin xyz=0 -0.5 0 rpy=0 0 0, axis 1 1 0, limit lower=-3.14159 upper=3.14159 effort=0.0 velocity=0.0
- added joint 4Link1_4Link2: type revolute, parent 4Link1, child 4Link2, origin xyz=0 -0.5 0 rpy=0 0 0, axis 1 1 0, limit lower=-3.14159 upper=3.14159 effort=0.0 velocity=0.0
- added joint 4Link2_4Link3: type revolute, parent 4Link2, child 4Link3, origin xyz=0 -0.5 0 rpy=0 0 0, axis 1 1 0, limit lower=-3.14159 upper=3.14159 effort=0.0 velocity=0.0
- added joint 4Link3_4Link4: type revolute, parent 4Link3, child 4Link4, origin xyz=0 -0.5 0 rpy=0 0 0, axis 1 1 0, limit lower=-3.14159 upper=3.14159 effort=0.0 velocity=0.0
- added joint 4Link4_4Link5: type revolute, parent 4Link4, child 4Link5, origin xyz=0 -0.5 0 rpy=0 0 0, axis 1 1 0, limit lower=-3.14159 upper=3.14159 effort=0.0 velocity=0.0
- added joint 4Link5_4Link6: type revolute, parent 4Link5, child 4Link6, origin xyz=0 -0.5 0 rpy=0 0 0, axis 1 1 0, limit lower=-3.14159 upper=3.14159 effort=0.0 velocity=0.0
- added joint 4Link6_4Link7: type revolute, parent 4Link6, child 4Link7, origin xyz=0 -0.5 0 rpy=0 0 0, axis 1 1 0, limit lower=-3.14159 upper=3.14159 effort=0.0 velocity=0.0
- added joint 4Link7_4Link8: type revolute, parent 4Link7, child 4Link8, origin xyz=0 -0.5 0 rpy=0 0 0, axis 1 1 0, limit lower=-3.14159 upper=3.14159 effort=0.0 velocity=0.0
- added joint 4Link8_4Link9: type revolute, parent 4Link8, child 4Link9, origin xyz=0 -0.5 0 rpy=0 0 0, axis 1 1 0, limit lower=-3.14159 upper=3.14159 effort=0.0 velocity=0.0
- added joint 4Link9_4Link10: type revolute, parent 4Link9, child 4Link10, origin xyz=0 -0.5 0 rpy=0 0 0, axis 1 1 0, limit lower=-3.14159 upper=3.14159 effort=0.0 velocity=0.0
- added joint 5Link0_5Link1: type revolute, parent 5Link0, child 5Link1, origin xyz=0 0.5 0 rpy=0 0 0, axis 1 1 0, limit lower=-3.14159 upper=3.14159 effort=0.0 velocity=0.0
- added joint 5Link10_5Link11: type revolute, parent 5Link10, child 5Link11, origin xyz=0 0.5 0 rpy=0 0 0, axis 1 1 0, limit lower=-3.14159 upper=3.14159 effort=0.0 velocity=0.0
- added joint 5Link11_5Link12: type revolute, parent 5Link11, child 5Link12, origin xyz=0 0.5 0 rpy=0 0 0, axis 1 1 0, limit lower=-3.14159 upper=3.14159 effort=0.0 velocity=0.0
- added joint 5Link12_5Link13: type revolute, parent 5Link12, child 5Link13, origin xyz=0 0.5 0 rpy=0 0 0, axis 1 1 0, limit lower=-3.14159 upper=3.14159 effort=0.0 velocity=0.0
- added joint 5Link13_5Link14: type revolute, parent 5Link13, child 5Link14, origin xyz=0 0.5 0 rpy=0 0 0, axis 1 1 0, limit lower=-3.14159 upper=3.14159 effort=0.0 velocity=0.0
- added joint 5Link14_5Link15: type revolute, parent 5Link14, child 5Link15, origin xyz=0 0.5 0 rpy=0 0 0, axis 1 1 0, limit lower=-3.14159 upper=3.14159 effort=0.0 velocity=0.0
- added joint 5Link15_5Link16: type revolute, parent 5Link15, child 5Link16, origin xyz=0 0.5 0 rpy=0 0 0, axis 1 1 0, limit lower=-3.14159 upper=3.14159 effort=0.0 velocity=0.0
- added joint 5Link16_5Link17: type revolute, parent 5Link16, child 5Link17, origin xyz=0 0.5 0 rpy=0 0 0, axis 1 1 0, limit lower=-3.14159 upper=3.14159 effort=0.0 velocity=0.0
- added joint 5Link1_5Link2: type revolute, parent 5Link1, child 5Link2, origin xyz=0 0.5 0 rpy=0 0 0, axis 1 1 0, limit lower=-3.14159 upper=3.14159 effort=0.0 velocity=0.0
- added joint 5Link2_5Link3: type revolute, parent 5Link2, child 5Link3, origin xyz=0 0.5 0 rpy=0 0 0, axis 1 1 0, limit lower=-3.14159 upper=3.14159 effort=0.0 velocity=0.0
- added joint 5Link3_5Link4: type revolute, parent 5Link3, child 5Link4, origin xyz=0 0.5 0 rpy=0 0 0, axis 1 1 0, limit lower=-3.14159 upper=3.14159 effort=0.0 velocity=0.0
- added joint 5Link4_5Link5: type revolute, parent 5Link4, child 5Link5, origin xyz=0 0.5 0 rpy=0 0 0, axis 1 1 0, limit lower=-3.14159 upper=3.14159 effort=0.0 velocity=0.0
- added joint 5Link5_5Link6: type revolute, parent 5Link5, child 5Link6, origin xyz=0 0.5 0 rpy=0 0 0, axis 1 1 0, limit lower=-3.14159 upper=3.14159 effort=0.0 velocity=0.0
- added joint 5Link6_5Link7: type revolute, parent 5Link6, child 5Link7, origin xyz=0 0.5 0 rpy=0 0 0, axis 1 1 0, limit lower=-3.14159 upper=3.14159 effort=0.0 velocity=0.0
- added joint 5Link7_5Link8: type revolute, parent 5Link7, child 5Link8, origin xyz=0 0.5 0 rpy=0 0 0, axis 1 1 0, limit lower=-3.14159 upper=3.14159 effort=0.0 velocity=0.0
- added joint 5Link8_5Link9: type revolute, parent 5Link8, child 5Link9, origin xyz=0 0.5 0 rpy=0 0 0, axis 1 1 0, limit lower=-3.14159 upper=3.14159 effort=0.0 velocity=0.0
- added joint 5Link9_5Link10: type revolute, parent 5Link9, child 5Link10, origin xyz=0 0.5 0 rpy=0 0 0, axis 1 1 0, limit lower=-3.14159 upper=3.14159 effort=0.0 velocity=0.0
- added joint Torso_4Link0: type revolute, parent Torso, child 4Link0, origin xyz=0.0 1.5 10.0 rpy=0 0 0, axis 1 1 0, limit lower=-3.14159 upper=3.14159 effort=0.0 velocity=0.0
- added joint Torso_5Link0: type revolute, parent Torso, child 5Link0, origin xyz=0.0 2.5 10.0 rpy=0 0 0, axis 1 1 0, limit lower=-3.14159 upper=3.14159 effort=0.0 velocity=0.0
