Commit message: etc

File: body.urdf (robot description, URDF)
Before this commit: robot robot, 94 links, 93 joints
Links:
- removed link 0Link10
- removed link 0Link11
- removed link 0Link12
- removed link 0Link13
- removed link 0Link14
- removed link 0Link15
- removed link 0Link5
- removed link 0Link6
- removed link 0Link7
- removed link 0Link8
- removed link 0Link9
- removed link 1Link10
- removed link 1Link11
- removed link 1Link12
- removed link 1Link13
- removed link 1Link14
- removed link 1Link15
- removed link 1Link16
- removed link 1Link4
- removed link 1Link5
- removed link 1Link6
- removed link 1Link7
- removed link 1Link8
- removed link 1Link9
- removed link 2Link10
- removed link 2Link11
- removed link 2Link12
- removed link 2Link13
- removed link 2Link14
- removed link 2Link2
- removed link 2Link3
- removed link 2Link4
- removed link 2Link5
- removed link 2Link6
- removed link 2Link7
- removed link 2Link8
- removed link 2Link9
- removed link 3Link10
- removed link 3Link11
- removed link 3Link3
- removed link 3Link4
- removed link 3Link5
- removed link 3Link6
- removed link 3Link7
- removed link 3Link8
- removed link 3Link9
- removed link 4Link10
- removed link 4Link11
- removed link 4Link12
- removed link 4Link13
- removed link 4Link14
- removed link 4Link4
- removed link 4Link5
- removed link 4Link6
- removed link 4Link7
- removed link 4Link8
- removed link 4Link9
- removed link 5Link10
- removed link 5Link11
- removed link 5Link12
- removed link 5Link13
- removed link 5Link14
- removed link 5Link15
- removed link 5Link16
- removed link 5Link17
- removed link 5Link3
- removed link 5Link4
- removed link 5Link5
- removed link 5Link6
- removed link 5Link7
- removed link 5Link8
- removed link 5Link9
- link 0Link0: geometry collision box size=0.5 0.5 0.5; visual box size=0.5 0.5 0.5
- link 0Link1: geometry collision box size=0.5 0.5 0.5; visual box size=0.5 0.5 0.5
- link 0Link2: geometry collision box size=0.5 0.5 0.5; visual box size=0.5 0.5 0.5
- link 0Link3: geometry collision box size=0.5 0.5 0.5; visual box size=0.5 0.5 0.5
- link 0Link4: geometry collision box size=0.5 0.5 0.5; visual box size=0.5 0.5 0.5
- link 1Link0: geometry collision box size=0.5 0.5 0.5; visual box size=0.5 0.5 0.5
- link 1Link1: geometry collision box size=0.5 0.5 0.5; visual box size=0.5 0.5 0.5
- link 1Link2: geometry collision box size=0.5 0.5 0.5; visual box size=0.5 0.5 0.5
- link 1Link3: geometry collision box size=0.5 0.5 0.5; visual box size=0.5 0.5 0.5
- link 2Link0: geometry collision box size=0.5 0.5 0.5; visual box size=0.5 0.5 0.5
- link 2Link1: geometry collision box size=0.5 0.5 0.5; visual box size=0.5 0.5 0.5
- link 3Link0: geometry collision box size=0.5 0.5 0.5; visual box size=0.5 0.5 0.5
- link 3Link1: geometry collision box size=0.5 0.5 0.5; visual box size=0.5 0.5 0.5
- link 3Link2: geometry collision box size=0.5 0.5 0.5; visual box size=0.5 0.5 0.5
- link 4Link0: geometry collision box size=0.5 0.5 0.5; visual box size=0.5 0.5 0.5
- link 4Link1: geometry collision box size=0.5 0.5 0.5; visual box size=0.5 0.5 0.5
- link 4Link2: geometry collision box size=0.5 0.5 0.5; visual box size=0.5 0.5 0.5
- link 4Link3: geometry collision box size=0.5 0.5 0.5; visual box size=0.5 0.5 0.5
- link 5Link0: geometry collision box size=0.5 0.5 0.5; visual box size=0.5 0.5 0.5
- link 5Link1: geometry collision box size=0.5 0.5 0.5; visual box size=0.5 0.5 0.5
- link 5Link2: geometry collision box size=0.5 0.5 0.5; visual box size=0.5 0.5 0.5
- link Torso: geometry collision box size=1.25 1.25 1.25; visual box size=1.25 1.25 1.25
Joints:
- removed joint 0Link10_0Link11
- removed joint 0Link11_0Link12
- removed joint 0Link12_0Link13
- removed joint 0Link13_0Link14
- removed joint 0Link14_0Link15
- removed joint 0Link4_0Link5
- removed joint 0Link5_0Link6
- removed joint 0Link6_0Link7
- removed joint 0Link7_0Link8
- removed joint 0Link8_0Link9
- removed joint 0Link9_0Link10
- removed joint 1Link10_1Link11
- removed joint 1Link11_1Link12
- removed joint 1Link12_1Link13
- removed joint 1Link13_1Link14
- removed joint 1Link14_1Link15
- removed joint 1Link15_1Link16
- removed joint 1Link3_1Link4
- removed joint 1Link4_1Link5
- removed joint 1Link5_1Link6
- removed joint 1Link6_1Link7
- removed joint 1Link7_1Link8
- removed joint 1Link8_1Link9
- removed joint 1Link9_1Link10
- removed joint 2Link10_2Link11
- removed joint 2Link11_2Link12
- removed joint 2Link12_2Link13
- removed joint 2Link13_2Link14
- removed joint 2Link1_2Link2
- removed joint 2Link2_2Link3
- removed joint 2Link3_2Link4
- removed joint 2Link4_2Link5
- removed joint 2Link5_2Link6
- removed joint 2Link6_2Link7
- removed joint 2Link7_2Link8
- removed joint 2Link8_2Link9
- removed joint 2Link9_2Link10
- removed joint 3Link10_3Link11
- removed joint 3Link2_3Link3
- removed joint 3Link3_3Link4
- removed joint 3Link4_3Link5
- removed joint 3Link5_3Link6
- removed joint 3Link6_3Link7
- removed joint 3Link7_3Link8
- removed joint 3Link8_3Link9
- removed joint 3Link9_3Link10
- removed joint 4Link10_4Link11
- removed joint 4Link11_4Link12
- removed joint 4Link12_4Link13
- removed joint 4Link13_4Link14
- removed joint 4Link3_4Link4
- removed joint 4Link4_4Link5
- removed joint 4Link5_4Link6
- removed joint 4Link6_4Link7
- removed joint 4Link7_4Link8
- removed joint 4Link8_4Link9
- removed joint 4Link9_4Link10
- removed joint 5Link10_5Link11
- removed joint 5Link11_5Link12
- removed joint 5Link12_5Link13
- removed joint 5Link13_5Link14
- removed joint 5Link14_5Link15
- removed joint 5Link15_5Link16
- removed joint 5Link16_5Link17
- removed joint 5Link2_5Link3
- removed joint 5Link3_5Link4
- removed joint 5Link4_5Link5
- removed joint 5Link5_5Link6
- removed joint 5Link6_5Link7
- removed joint 5Link7_5Link8
- removed joint 5Link8_5Link9
- removed joint 5Link9_5Link10
